File: hardware/v0.1a/icebreaker.sch (KiCad schematic (older format))
At the start: 108 parts, among them J1 Jumper, J10 Jumper, J11 Jumper, J12 Jumper, J13 Jumper, J14 Jumper, J15 Jumper, J16 Jumper, J17 Jumper, J18 Jumper, J19 Jumper, J2 Jumper, J20 Flash, J21 PMOD_1A, J22 PMOD_1B, J23 PMOD_2H, J24 PMOD_2P, J25 RGB Led, J26 5V AUX, J27 5V AUX, J3 Jumper, J4 Jumper, J5 Jumper, J6 Jumper, J7 Jumper, J8 Jumper, J9 Jumper, P1 pkl_USB_OTG, SW1 TACT, SW2 TACT, SW3 TACT, SW4 TACT, U1 93C46B-SOT-23-6, U2 3.3V, U3 1V2, U4 FT2232H, U5 W25Q, U6 ICE5LP4K-SG48, X1 12MHz

Commit message: Update the v0.1a schematic to use up to date libraries.
Parts:
- J20: symbol conn:Conn_01x07 -> Connector_Generic:Conn_01x07
- J21, J22, J23, J24: symbol conn:Conn_02x06_Top_Bottom -> Connector_Generic:Conn_02x06_Top_Bottom
- J25: symbol conn:Conn_02x04_Odd_Even -> Connector_Generic:Conn_02x04_Odd_Even
- J26, J27: symbol conn:Conn_02x01 -> Connector_Generic:Conn_02x01
Changed lines of the file:
@@
 	10700 2150 10700 2300
 $Comp
-L conn:Conn_02x06_Top_Bottom J21
+L Connector_Generic:Conn_02x06_Top_Bottom J21
 U 1 1 5B1E5C63
 P 12400 2400
@@
 F 2 "Socket_Strips:Socket_Strip_Angled_2x06" H 12400 2400 50  0001 C CNN
 F 3 "~" H 12400 2400 50  0001 C CNN
-F 4 "ANY" H 12400 2400 50  0001 C CNN "Source"
-F 5 "conn-th-01in-6-2-rec-ra" H 0   0   50  0001 C CNN "Key"
+F 4 "conn-th-01in-6-2-rec-ra" H 0   0   50  0001 C CNN "Key"
+F 5 "ANY" H 12400 2400 50  0001 C CNN "Source"
 	1    12400 2400
 	1    0    0    -1
 $EndComp
 $Comp
-L conn:Conn_02x06_Top_Bottom J22
+L Connector_Generic:Conn_02x06_Top_Bottom J22
 U 1 1 5B1E5EFC
 P 12400 4100
@@
 F 2 "Socket_Strips:Socket_Strip_Angled_2x06" H 12400 4100 50  0001 C CNN
 F 3 "~" H 12400 4100 50  0001 C CNN
-F 4 "ANY" H 12400 4100 50  0001 C CNN "Source"
-F 5 "conn-th-01in-6-2-rec-ra" H 0   0   50  0001 C CNN "Key"
+F 4 "conn-th-01in-6-2-rec-ra" H 0   0   50  0001 C CNN "Key"
+F 5 "ANY" H 12400 4100 50  0001 C CNN "Source"
 	1    12400 4100
 	1    0    0    -1
@@
 $EndComp
 $Comp
-L conn:Conn_02x04_Odd_Even J25
+L Connector_Generic:Conn_02x04_Odd_Even J25
 U 1 1 5B43F731
 P 14900 8700
@@
 F 2 "Pin_Headers:Pin_Header_Straight_2x04" H 14900 8700 50  0001 C CNN
 F 3 "~" H 14900 8700 50  0001 C CNN
-F 4 "ANY" H 14900 8700 50  0001 C CNN "Source"
-F 5 "conn-th-01in-4-2-hdr" H 0   0   50  0001 C CNN "Key"
+F 4 "conn-th-01in-4-2-hdr" H 0   0   50  0001 C CNN "Key"
+F 5 "ANY" H 14900 8700 50  0001 C CNN "Source"
 	1    14900 8700
 	1    0    0    -1
@@
 Connection ~ 8500 5500
 $Comp
-L conn:Conn_02x06_Top_Bottom J23
+L Connector_Generic:Conn_02x06_Top_Bottom J23
 U 1 1 5BFA913D
 P 12400 5600
@@
 F 2 "Socket_Strips:Socket_Strip_Straight_2x06" H 12400 5600 50  0001 C CNN
 F 3 "~" H 12400 5600 50  0001 C CNN
-F 4 "ANY" H 12400 5600 50  0001 C CNN "Source"
-F 5 "conn-th-01in-6-2-rec-ra" H 0   0   50  0001 C CNN "Key"
+F 4 "conn-th-01in-6-2-rec-ra" H 0   0   50  0001 C CNN "Key"
+F 5 "ANY" H 12400 5600 50  0001 C CNN "Source"
 	1    12400 5600
 	1    0    0    -1
 $EndComp
 $Comp
-L conn:Conn_02x06_Top_Bottom J24
+L Connector_Generic:Conn_02x06_Top_Bottom J24
 U 1 1 5BFA93A4
 P 14050 5600
@@
 F 2 "Pin_Headers:Pin_Header_Straight_2x06" H 14050 5600 50  0001 C CNN
 F 3 "~" H 14050 5600 50  0001 C CNN
-F 4 "ANY" H 14050 5600 50  0001 C CNN "Source"
-F 5 "conn-th-01in-6-2-hdr-ra" H 0   0   50  0001 C CNN "Key"
+F 4 "conn-th-01in-6-2-hdr-ra" H 0   0   50  0001 C CNN "Key"
+F 5 "ANY" H 14050 5600 50  0001 C CNN "Source"
 	1    14050 5600
 	1    0    0    -1
@@
 FLASH_~HLD~/~RST~/IO3
 $Comp
-L conn:Conn_01x07 J20
+L Connector_Generic:Conn_01x07 J20
 U 1 1 5EB92B77
 P 11250 8050
@@
 F 2 "Pin_Headers:Pin_Header_Straight_1x07" H 11250 8050 50  0001 C CNN
 F 3 "~" H 11250 8050 50  0001 C CNN
-F 4 "ANY" H 11250 8050 50  0001 C CNN "Source"
-F 5 "conn-th-01in-7-1-hdr" H 0   0   50  0001 C CNN "Key"
+F 4 "conn-th-01in-7-1-hdr" H 0   0   50  0001 C CNN "Key"
+F 5 "ANY" H 11250 8050 50  0001 C CNN "Source"
 	1    11250 8050
 	1    0    0    -1
@@
 $EndComp
 $Comp
-L conn:Conn_02x01 J26
+L Connector_Generic:Conn_02x01 J26
 U 1 1 5A936954
 P 12400 3300
@@
 F 2 "Pin_Headers:Pin_Header_Straight_2x01" H 12400 3300 50  0001 C CNN
 F 3 "~" H 12400 3300 50  0001 C CNN
-F 4 "ANY" H 12400 3300 50  0001 C CNN "Source"
-F 5 "conn-th-01in-2-1-hdr" H 0   0   50  0001 C CNN "Key"
+F 4 "conn-th-01in-2-1-hdr" H 0   0   50  0001 C CNN "Key"
+F 5 "ANY" H 12400 3300 50  0001 C CNN "Source"
 	1    12400 3300
 	1    0    0    -1
@@
 $EndComp
 $Comp
-L conn:Conn_02x01 J27
+L Connector_Generic:Conn_02x01 J27
 U 1 1 5A5CE3A7
 P 12400 6550
@@
 F 2 "Pin_Headers:Pin_Header_Straight_2x01" H 12400 6550 50  0001 C CNN
 F 3 "~" H 12400 6550 50  0001 C CNN
-F 4 "ANY" H 12400 6550 50  0001 C CNN "Source"
-F 5 "conn-th-01in-2-1-hdr" H 0   0   50  0001 C CNN "Key"
+F 4 "conn-th-01in-2-1-hdr" H 0   0   50  0001 C CNN "Key"
+F 5 "ANY" H 12400 6550 50  0001 C CNN "Source"
 	1    12400 6550
 	1    0    0    -1
