File: hardware/bitsy-v0.1a/icebreaker-bitsy.sch (KiCad schematic (older format))
At the start: 92 parts, among them J1 Conn_01x01, J10 Conn_01x01, J11 Conn_01x01, J12 Conn_01x01, J13 Conn_01x01, J14 Jumper, J15 Jumper, J16 Jumper, J17 Jumper, J18 Jumper, J19 Jumper, J2 Conn_01x01, J20 Conn_01x01, J21 Conn_01x01, J22 Conn_01x01, J23 Conn_01x01, J24 Conn_01x01, J25 Conn_01x01, J26 Conn_01x01, J27 Conn_01x01, J28 Conn_01x01, J29 Conn_01x01, J3 Conn_01x01, J30 Conn_01x01, J31 Conn_01x01, J32 Conn_01x01, J33 Conn_01x01, J34 Conn_01x01, J35 Conn_01x01, J36 Conn_01x01, J37 Conn_01x01, J4 Conn_01x01, J41 Conn_01x01, J42 Conn_01x01, J43 Conn_01x01, J44 Conn_01x01, J45 Conn_01x01, J46 Conn_01x01, J47 Conn_01x01, J48 Conn_01x01, J49 Conn_01x01, J5 Conn_01x01, J6 Conn_01x01, J7 Conn_01x01, J8 Conn_01x01, J9 Conn_01x01, P1 pkl_USB_OTG, SW1 TACT, U2 3.3V, U3 1V2, U5 W25Q, U6 ICE5LP4K-SG48, X1 12MHz

Commit message: Schematic cleanup and minor improvements.
Added ESD protection on the USB interface, added +5V VIN Jumper.
Parts:
- added J38: Jumper, pkl_jumpers:J_0603, symbol pkl_misc:Jumper
- added U1: USBLC6-2, pkl_housings_sot:SOT-666, symbol pkl_misc:USBLC6-2
- P1: value pkl_USB_OTG -> USB_OTG
Connections:
- net labels added: iUD+, iUD-
- wire segments 299 -> 315
Other:
- note added: "1V2 VReg"
- note added: "3V3 VReg"
- note added: "For programming iCE FPGA:\n* cut traces connecting J15 and J16 pads.\n* Short the pads 1 and 2 together of the J15 and J16\nFor programming Flash reverse the operations."
- note added: "iCE FPGA Flash\n& Prog Pins"
- note removed: "1V2 VReg Device"
- note removed: "3V3 VReg Device"
- note removed: "For programming iCE cut traces connecting J15 and J16 pads.\nShort the pads 1 and 2 together of the J15 and J16 respectively.\nFor programming Flash reverse the operations."

Commit message: Adjusted USB resistor values based on Luke Valenty suggestions.
Thanks @tinyfpga ! :D
Parts:
- R2: value 15k -> 1k5; Key res-0402-10k -> res-0402-1k5
- R4, R6: value 68E -> 22E; Key res-0402-10k -> res-0402-22
Other:
- note added: "Using same values\nas STM32F1 spec"
- note removed: "Really 68?\nNot 22?"
Changed lines of the file:
@@
 P 3800 1100
 F 0 "R2" V 3700 1050 50  0000 C CNN
-F 1 "15k" V 3700 1250 50  0000 C CNN
+F 1 "1k5" V 3700 1250 50  0000 C CNN
 F 2 "pkl_dipol:R_0402" H 3859 1007 60  0001 L CNN
 F 3 "" H 3800 1100 60  0000 C CNN
-F 4 "res-0402-10k" H -7400 -4300 50  0001 C CNN "Key"
+F 4 "res-0402-1k5" H -7400 -4300 50  0001 C CNN "Key"
 F 5 "ANY" H 3800 1100 50  0001 C CNN "Source"
 	1    3800 1100
@@
 P 4100 1300
 F 0 "R4" V 3901 1300 50  0000 C CNN
-F 1 "68E" V 3994 1300 50  0000 C CNN
+F 1 "22E" V 3994 1300 50  0000 C CNN
 F 2 "pkl_dipol:R_0402" H 4159 1207 60  0001 L CNN
 F 3 "" H 4100 1300 60  0000 C CNN
-F 4 "res-0402-10k" H -7100 -4100 50  0001 C CNN "Key"
+F 4 "res-0402-22" H -7100 -4100 50  0001 C CNN "Key"
 F 5 "ANY" H 4100 1300 50  0001 C CNN "Source"
 	1    4100 1300
@@
 P 4100 1400
 F 0 "R6" V 4205 1400 50  0000 C CNN
-F 1 "68E" V 4298 1400 50  0000 C CNN
+F 1 "22E" V 4298 1400 50  0000 C CNN
 F 2 "pkl_dipol:R_0402" H 4159 1307 60  0001 L CNN
 F 3 "" H 4100 1400 60  0000 C CNN
-F 4 "res-0402-10k" H -7100 -4000 50  0001 C CNN "Key"
+F 4 "res-0402-22" H -7100 -4000 50  0001 C CNN "Key"
 F 5 "ANY" H 4100 1400 50  0001 C CNN "Source"
 	1    4100 1400
 	0    1    1    0
 $EndComp
-Text Notes 3950 1800 0    50   ~ 0
-Really 68?\nNot 22?
+Text Notes 3800 1800 0    50   ~ 0
+Using same values\nas STM32F1 spec
 Wire Wire Line
 	4200 1300 4300 1300

Commit message: Minor cleanups, ready to order prototypes! :D
Parts:
- C35: Key (none) -> cap-cer-0402-10n
- D2: Key diode-shottky-0603 -> diode-schottky-0603
- U1: Key (none) -> tvs-diode-sot666
Changed lines of the file:
@@
 F 2 "pkl_dipol:D_0603" V 6750 4800 60  0001 C CNN
 F 3 "" V 6750 4800 60  0000 C CNN
-F 4 "ANY" H 6750 4800 50  0001 C CNN "Source"
-F 5 "diode-shottky-0603" H -1400 -1000 50  0001 C CNN "Key"
+F 4 "diode-schottky-0603" H -1400 -1000 50  0001 C CNN "Key"
+F 5 "ANY" H 6750 4800 50  0001 C CNN "Source"
 	1    6750 4800
 	1    0    0    -1
@@
 F 2 "pkl_dipol:C_0402" H 7042 4907 60  0001 L CNN
 F 3 "" H 6950 5000 60  0000 C CNN
-F 4 "ANY" H 6950 5000 50  0001 C CNN "Source"
+F 4 "cap-cer-0402-10n" H 6950 5000 50  0001 C CNN "Key"
+F 5 "ANY" H 6950 5000 50  0001 C CNN "Source"
 	1    6950 5000
 	-1   0    0    -1
@@
 F 2 "pkl_housings_sot:SOT-666" H 2600 1585 60  0001 C CNN
 F 3 "" H 2600 1300 60  0000 C CNN
-F 4 "ANY" H 2600 1300 50  0001 C CNN "Source"
+F 4 "tvs-diode-sot666" H 2600 1300 50  0001 C CNN "Key"
+F 5 "ANY" H 2600 1300 50  0001 C CNN "Source"
 	1    2600 1300
 	1    0    0    -1

Commit message: Added pinout information and updated schematic.
Connections:
- net labels added: IOT_36B
- net labels removed: IOT_36b
Changed lines of the file:
@@
 	9200 2900 9800 2900
 Text Label 9400 1500 0    50   ~ 0
-IOT_36b
+IOT_36B
 Text Label 9400 1600 0    50   ~ 0
 IOT_37A

Commit message: Update the bitsy-v0.1a schematic to use up to date libraries.
Parts:
- J1, J10, J11, J12, J13, J2, J20, J21, J22, J23, J24, J25, J26, J27, J28, J29, J3, J30, J31, J32, J33, J34, J35, J36, J37, J4, J41, J42, J43, J44, J45, J46, J47, J48, J49, J5, J6, J7, J8, J9: symbol conn:Conn_01x01 -> Connector_Generic:Conn_01x01
Changed lines of the file:
@@
 	-1   0    0    1
 $EndComp
-Wire Wire Line
-	1950 3150 2050 3150
 $Comp
 L pkl_device:pkl_R_Small R7
@@
 	1    0    0    -1
 $EndComp
-Wire Wire Line
-	1150 3050 1050 3050
-Wire Wire Line
-	1050 3050 1050 2950
 $Comp
 L power:+3V3 #PWR03
@@
 	1    0    0    -1
 $EndComp
-Wire Wire Line
-	1150 3150 1050 3150
-Wire Wire Line
-	1050 3150 1050 3450
 $Comp
 L pkl_device:pkl_C_Small C4
@@
 	-1   0    0    -1
 $EndComp
-Wire Wire Line
-	850  3350 850  3450
-Wire Wire Line
-	850  3150 850  3050
-Wire Wire Line
-	850  3050 1050 3050
-Connection ~ 1050 3050
 $Comp
 L power:GND #PWR05
@@
 	1    0    0    -1
 $EndComp
-Wire Wire Line
-	850  3450 950  3450
-Wire Wire Line
-	950  3450 950  3550
-Connection ~ 950  3450
-Wire Wire Line
-	950  3450 1050 3450
-Wire Wire Line
-	2250 3150 2450 3150
-Wire Wire Line
-	2450 2950 2450 3150
 Text Notes 1950 3350 0    50   ~ 0
 10k or less
@@
 Text Notes 550  5050 0    50   ~ 0
 Enable Delay\n~~0.001s\nShould enable\nafter 1v2 rail\n(Test!!!)
-Wire Wire Line
-	1950 3050 2050 3050
 $Comp
 L pkl_device:pkl_R_Small R2
@@
 USB_P
 $Comp
-L conn:Conn_01x01 J21
+L Connector_Generic:Conn_01x01 J21
 U 1 1 5ACEE8F6
 P 6600 5800
@@
 $EndComp
 $Comp
-L conn:Conn_01x01 J22
+L Connector_Generic:Conn_01x01 J22
 U 1 1 5ACEF407
 P 6600 5900
@@
 $EndComp
 $Comp
-L conn:Conn_01x01 J23
+L Connector_Generic:Conn_01x01 J23
 U 1 1 5ACEF48F
 P 6600 6000
@@
 $EndComp
 $Comp
-L conn:Conn_01x01 J24
+L Connector_Generic:Conn_01x01 J24
 U 1 1 5ACEF519
 P 6600 6100
@@
 $EndComp
 $Comp
-L conn:Conn_01x01 J25
+L Connector_Generic:Conn_01x01 J25
 U 1 1 5ACEF5A5
 P 6600 6200
@@
 $EndComp
 $Comp
-L conn:Conn_01x01 J26
+L Connector_Generic:Conn_01x01 J26
 U 1 1 5ACEF633
 P 6600 6300
@@
 $EndComp
 $Comp
-L conn:Conn_01x01 J27
+L Connector_Generic:Conn_01x01 J27
 U 1 1 5ACEF6C3
 P 6600 6400
@@
 $EndComp
 $Comp
-L conn:Conn_01x01 J28
+L Connector_Generic:Conn_01x01 J28
 U 1 1 5ACEF755
 P 6600 6500
@@
 	6400 6500 6300 6500
 $Comp
-L conn:Conn_01x01 J7
+L Connector_Generic:Conn_01x01 J7
 U 1 1 5AD40D83
 P 6500 1500
@@
 $EndComp
 $Comp
-L conn:Conn_01x01 J8
+L Connector_Generic:Conn_01x01 J8
 U 1 1 5AD4158F
 P 6500 1600
@@
 $EndComp
 $Comp
-L conn:Conn_01x01 J9
+L Connector_Generic:Conn_01x01 J9
 U 1 1 5AD41627
 P 6500 1700
@@
 $EndComp
 $Comp
-L conn:Conn_01x01 J10
+L Connector_Generic:Conn_01x01 J10
 U 1 1 5AD416C1
 P 6500 1800
@@
 $EndComp
 $Comp
-L conn:Conn_01x01 J11
+L Connector_Generic:Conn_01x01 J11
 U 1 1 5AD4175D
 P 6500 1900
@@
 $EndComp
 $Comp
-L conn:Conn_01x01 J12
+L Connector_Generic:Conn_01x01 J12
 U 1 1 5AD417FB
 P 6500 2000
@@
 $EndComp
 $Comp
-L conn:Conn_01x01 J13
+L Connector_Generic:Conn_01x01 J13
 U 1 1 5AD4189B
 P 6500 2100
@@
 $EndComp
 $Comp
-L conn:Conn_01x01 J20
+L Connector_Generic:Conn_01x01 J20
 U 1 1 5AD4193D
 P 6500 2200
@@
 IOB_9B
 $Comp
-L conn:Conn_01x01 J29
+L Connector_Generic:Conn_01x01 J29
 U 1 1 5AE1DB99
 P 10000 1500
@@
 $EndComp
 $Comp
-L conn:Conn_01x01 J30
+L Connector_Generic:Conn_01x01 J30
 U 1 1 5AE1E029
 P 10000 1600
@@
 $EndComp
 $Comp
-L conn:Conn_01x01 J31
+L Connector_Generic:Conn_01x01 J31
 U 1 1 5AE1E0D1
 P 10000 1700
@@
 $EndComp
 $Comp
-L conn:Conn_01x01 J32
+L Connector_Generic:Conn_01x01 J32
 U 1 1 5AE1E17B
 P 10000 1800
@@
 $EndComp
 $Comp
-L conn:Conn_01x01 J33
+L Connector_Generic:Conn_01x01 J33
 U 1 1 5AE1E227
 P 10000 1900
@@
 $EndComp
 $Comp
-L conn:Conn_01x01 J34
+L Connector_Generic:Conn_01x01 J34
 U 1 1 5AE1E2D5
 P 10000 2000
@@
 $EndComp
 $Comp
-L conn:Conn_01x01 J35
+L Connector_Generic:Conn_01x01 J35
 U 1 1 5AE1E385
 P 10000 2100
@@
 $EndComp
 $Comp
-L conn:Conn_01x01 J37
+L Connector_Generic:Conn_01x01 J37
 U 1 1 5AE1E437
 P 10000 2500
@@
 $EndComp
 $Comp
-L conn:Conn_01x01 J41
+L Connector_Generic:Conn_01x01 J41
 U 1 1 5AE1E71F
 P 10000 2900
@@
 $EndComp
 $Comp
-L conn:Conn_01x01 J42
+L Connector_Generic:Conn_01x01 J42
 U 1 1 5AE1E7DB
 P 10000 3000
@@
 $EndComp
 $Comp
-L conn:Conn_01x01 J43
+L Connector_Generic:Conn_01x01 J43
 U 1 1 5AE1E899
 P 10000 3100
@@
 $EndComp
 $Comp
-L conn:Conn_01x01 J36
+L Connector_Generic:Conn_01x01 J36
 U 1 1 5AE5210D
 P 10000 2200
@@
 USB_N
 $Comp
-L conn:Conn_01x01 J44
+L Connector_Generic:Conn_01x01 J44
 U 1 1 5AECDDB7
 P 10000 3500
@@
 $EndComp
 $Comp
-L conn:Conn_01x01 J45
+L Connector_Generic:Conn_01x01 J45
 U 1 1 5AECDEA1
 P 10000 3600
@@
 $EndComp
 $Comp
-L conn:Conn_01x01 J49
+L Connector_Generic:Conn_01x01 J49
 U 1 1 5AECDF67
 P 10200 4000
@@
 $EndComp
 $Comp
-L conn:Conn_01x01 J46
+L Connector_Generic:Conn_01x01 J46
 U 1 1 5AECE05B
 P 10000 4200
@@
 $EndComp
 $Comp
-L conn:Conn_01x01 J47
+L Connector_Generic:Conn_01x01 J47
 U 1 1 5AECE13D
 P 10000 4300
@@
 $EndComp
 $Comp
-L conn:Conn_01x01 J48
+L Connector_Generic:Conn_01x01 J48
 U 1 1 5AECE209
 P 10000 4400
@@
 USB
 $Comp
-L conn:Conn_01x01 J1
+L Connector_Generic:Conn_01x01 J1
 U 1 1 5B1151BE
 P 700 6200
@@
 $EndComp
 $Comp
-L conn:Conn_01x01 J2
+L Connector_Generic:Conn_01x01 J2
 U 1 1 5B14536A
 P 700 6300
@@
 $EndComp
 $Comp
-L conn:Conn_01x01 J3
+L Connector_Generic:Conn_01x01 J3
 U 1 1 5B1A6195
 P 700 6400
@@
 $EndComp
 $Comp
-L conn:Conn_01x01 J4
+L Connector_Generic:Conn_01x01 J4
 U 1 1 5B1A6265
 P 700 6500
@@
 $EndComp
 $Comp
-L conn:Conn_01x01 J5
+L Connector_Generic:Conn_01x01 J5
 U 1 1 5B1A6337
 P 700 6600
@@
 $EndComp
 $Comp
-L conn:Conn_01x01 J6
+L Connector_Generic:Conn_01x01 J6
 U 1 1 5B1A640B
 P 700 6700
@@
 Wire Notes Line
 	4700 5700 4700 7700
+Wire Wire Line
+	2450 2950 2450 3150
+Wire Wire Line
+	2250 3150 2450 3150
+Wire Wire Line
+	1950 3150 2050 3150
+Wire Wire Line
+	1950 3050 2050 3050
+Wire Wire Line
+	1050 3050 1050 2950
+Wire Wire Line
+	1150 3050 1050 3050
+Connection ~ 1050 3050
+Wire Wire Line
+	850  3050 1050 3050
+Wire Wire Line
+	850  3150 850  3050
+Wire Wire Line
+	850  3350 850  3450
+Wire Wire Line
+	950  3450 950  3550
+Wire Wire Line
+	850  3450 950  3450
+Connection ~ 950  3450
+Wire Wire Line
+	950  3450 1050 3450
+Wire Wire Line
+	1050 3150 1050 3450
+Wire Wire Line
+	1150 3150 1050 3150
 $EndSCHEMATC
