File: hardware/v0.2a/icebreaker.kicad_pcb (KiCad board)
At the start: 4 copper layers, 73 x 37 mm, 121 parts, among them J1 Jumper, J10 Jumper, J11 Jumper, J12 Jumper, J13 Jumper, J14 Jumper, J15 Jumper, J16 Jumper, J17 Jumper, J18 Jumper, J19 Jumper, J2 Jumper, J20 Flash, J21 PMOD_1A, J22 PMOD_1B, J23 PMOD_2H, J24 PMOD_2P, J25 RGB Led, J26 5V AUX, J27 5V AUX, J3 Jumper, J4 Jumper, J5 Jumper, J6 Jumper, J7 Jumper, J8 Jumper, J9 Jumper, P1 pkl_USB_OTG, SW1 TACT, SW2 TACT, SW3 TACT, SW4 TACT, U1 93C46B-SOT-23-6, U2 3.3V, U3 1V2, U4 FT2232H, U5 W25Q, U6 ICE5LP4K-SG48, U7 12MHz

Commit message: Added USB signal pads.
These pads can be used for testing, debugging as well as hard wiring a
usb extension cable.
Parts:
- added P2: UP, pkl_pads:PAD_SMD_1x2.65, B.Cu at (31.8, 43.7)
- added P3: UP, pkl_pads:PAD_SMD_1x2.65, B.Cu at (31.8, 46.2)
- added P4: UP, pkl_pads:PAD_SMD_1x2.65, B.Cu at (31.8, 48.8)
- added P5: UP, pkl_pads:PAD_SMD_1x2.65, B.Cu at (31.8, 51.3)
Routing:
- net Net-(P1-Pad3): track 5.65 -> 8.51 mm, vias 0 -> 1
- net Net-(P1-Pad2): track 5.64 -> 8.48 mm, vias 0 -> 1
- net +5V: track 147.1 -> 149.6 mm
- net GND: track 10.5 -> 12.8 mm, vias 21 -> 22
Changed lines of the file:
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@@
     (thickness 1.6)
     (drawings 95)
-    (tracks 1380)
+    (tracks 1400)
     (zones 0)
-    (modules 121)
+    (modules 125)
     (nets 125)
   )
@@
   )
   (setup
-    (last_trace_width 0.3)
+    (last_trace_width 0.15)
     (user_trace_width 0.2)
     (user_trace_width 0.3)
@@
     (mod_text_size 1 1)
     (mod_text_width 0.15)
-    (pad_size 2.225 2.225)
+    (pad_size 2.65 1)
     (pad_drill 0)
     (pad_to_mask_clearance 0.05)
@@
     (add_net "Net-(U7-Pad2)")
   )
+  (module pkl_pads:PAD_SMD_1x2.65 (layer B.Cu)
+    (at 31.84 51.31)
+    (fp_text reference P5 (at 0 -2.5) (layer B.Fab) hide
+      (effects (font (size 1 1) (thickness 0.15)) (justify mirror))
+    )
+    (fp_text value UP (at 0 2.2) (layer B.Fab) hide
+      (effects (font (size 1 1) (thickness 0.15)) (justify mirror))
+    )
+    (pad 1 smd roundrect (at 0 0) (size 2.65 1) (layers B.Cu B.Mask)(roundrect_rratio 0.25)
+      (net 28 GND))
+  )
+  (module pkl_pads:PAD_SMD_1x2.65 (layer B.Cu)
+    (at 31.84 43.69)
+    (fp_text reference P2 (at 0 -2.5) (layer B.Fab) hide
+      (effects (font (size 1 1) (thickness 0.15)) (justify mirror))
+    )
+    (fp_text value UP (at 0 2.2) (layer B.Fab) hide
+      (effects (font (size 1 1) (thickness 0.15)) (justify mirror))
+    )
+    (pad 1 smd roundrect (at 0 0) (size 2.65 1) (layers B.Cu B.Mask)(roundrect_rratio 0.25)
+      (net 34 +5V))
+  )
+  (module pkl_pads:PAD_SMD_1x2.65 (layer B.Cu)
+    (at 31.84 46.23)
+    (fp_text reference P3 (at 0 -2.5) (layer B.Fab) hide
+      (effects (font (size 1 1) (thickness 0.15)) (justify mirror))
+    )
+    (fp_text value UP (at 0 2.2) (layer B.Fab) hide
+      (effects (font (size 1 1) (thickness 0.15)) (justify mirror))
+    )
+    (pad 1 smd roundrect (at 0 0) (size 2.65 1) (layers B.Cu B.Mask)(roundrect_rratio 0.25)
+      (net 44 "Net-(P1-Pad2)"))
+  )
+  (module pkl_pads:PAD_SMD_1x2.65 (layer B.Cu)
+    (at 31.84 48.77)
+    (fp_text reference P4 (at 0 -2.5) (layer B.Fab) hide
+      (effects (font (size 1 1) (thickness 0.15)) (justify mirror))
+    )
+    (fp_text value UP (at 0 2.2) (layer B.Fab) hide
+      (effects (font (size 1 1) (thickness 0.15)) (justify mirror))
+    )
+    (pad 1 smd roundrect (at 0 0) (size 2.65 1) (layers B.Cu B.Mask)(roundrect_rratio 0.25)
+      (net 45 "Net-(P1-Pad3)"))
+  )
   (module pkl_dipol:R_Array_Convex_4x0402 (layer F.Cu)
     (at 57.105546 43.866206 45)
@@
   (segment (start 65.9 51.553554) (end 65.9 52.56066) (width 0.15) (layer F.Cu) (net 27))
   (segment (start 65.9 52.56066) (end 66.133794 52.794454) (width 0.15) (layer F.Cu) (net 27))
+  (segment (start 34.175 48.8) (end 33.4 48.8) (width 0.3) (layer F.Cu) (net 28))
+  (segment (start 32.7 49.5) (end 32.7 50) (width 0.3) (layer F.Cu) (net 28))
+  (via (at 32.7 50) (size 0.5) (drill 0.3) (layers F.Cu B.Cu) (net 28))
+  (segment (start 33.4 48.8) (end 32.7 49.5) (width 0.3) (layer F.Cu) (net 28))
   (via (at 71.5 50) (size 0.5) (drill 0.3) (layers F.Cu B.Cu) (net 28))
   (via (at 69.1 52.4) (size 0.5) (drill 0.3) (layers F.Cu B.Cu) (net 28))
@@
   (segment (start 63.013173 43.504847) (end 63.140124 43.377896) (width 0.15) (layer F.Cu) (net 32))
   (segment (start 45.600011 40.299989) (end 59.324268 40.299989) (width 0.15) (layer B.Cu) (net 32))
+  (segment (start 32.7 45) (end 32.7 44.55) (width 0.3) (layer B.Cu) (net 34))
+  (segment (start 32.7 44.55) (end 31.84 43.69) (width 0.3) (layer B.Cu) (net 34))
+  (segment (start 34.175 46.2) (end 33.4 46.2) (width 0.3) (layer F.Cu) (net 34))
+  (segment (start 33.4 46.2) (end 32.7 45.5) (width 0.3) (layer F.Cu) (net 34))
+  (segment (start 32.7 45.5) (end 32.7 45) (width 0.3) (layer F.Cu) (net 34))
+  (segment (start 32 65.4) (end 30.6 64) (width 0.3) (layer In2.Cu) (net 34))
+  (segment (start 30.6 47.1) (end 32.4 45.3) (width 0.3) (layer In2.Cu) (net 34))
+  (segment (start 30.6 64) (end 30.6 47.1) (width 0.3) (layer In2.Cu) (net 34))
+  (segment (start 40.1 65.4) (end 32 65.4) (width 0.3) (layer In2.Cu) (net 34))
+  (segment (start 32.4 45.3) (end 32.7 45) (width 0.3) (layer In2.Cu) (net 34))
+  (segment (start 55.1 33.53) (end 53.63 33.53) (width 0.3) (layer In2.Cu) (net 34))
+  (segment (start 52.6 32.5) (end 52.6 30.7) (width 0.3) (layer In2.Cu) (net 34))
+  (segment (start 52.6 30.7) (end 51.3 29.4) (width 0.3) (layer In2.Cu) (net 34))
+  (segment (start 53.63 33.53) (end 52.6 32.5) (width 0.3) (layer In2.Cu) (net 34))
+  (segment (start 30.6 42.9) (end 32.7 45) (width 0.3) (layer In2.Cu) (net 34))
+  (segment (start 30.6 31) (end 30.6 42.9) (width 0.3) (layer In2.Cu) (net 34))
+  (segment (start 32.2 29.4) (end 30.6 31) (width 0.3) (layer In2.Cu) (net 34))
+  (segment (start 51.3 29.4) (end 32.2 29.4) (width 0.3) (layer In2.Cu) (net 34))
+  (via (at 32.7 45) (size 0.5) (drill 0.3) (layers F.Cu B.Cu) (net 34))
   (segment (start 63.366726 51.1416) (end 68.5 56.274874) (width 0.15) (layer F.Cu) (net 39))
   (segment (start 68.5 56.274874) (end 68.5 59.1) (width 0.15) (layer F.Cu) (net 39))
+  (via (at 32.900002 47.15) (size 0.5) (drill 0.3) (layers F.Cu B.Cu) (net 44))
+  (segment (start 31.84 46.23) (end 32.76 47.15) (width 0.15) (layer B.Cu) (net 44))
+  (segment (start 34.175 46.85) (end 33.200002 46.85) (width 0.15) (layer F.Cu) (net 44))
+  (segment (start 32.76 47.15) (end 32.900002 47.15) (width 0.15) (layer B.Cu) (net 44))
+  (segment (start 33.200002 46.85) (end 32.900002 47.15) (width 0.15) (layer F.Cu) (net 44))
+  (segment (start 32.76 47.85) (end 32.9 47.85) (width 0.15) (layer B.Cu) (net 45))
+  (segment (start 33.999998 47.675002) (end 33.074998 47.675002) (width 0.15) (layer F.Cu) (net 45))
+  (via (at 32.9 47.85) (size 0.5) (drill 0.3) (layers F.Cu B.Cu) (net 45))
+  (segment (start 34.175 47.5) (end 33.999998 47.675002) (width 0.15) (layer F.Cu) (net 45))
+  (segment (start 33.074998 47.675002) (end 32.9 47.85) (width 0.15) (layer F.Cu) (net 45))
+  (segment (start 31.84 48.77) (end 32.76 47.85) (width 0.15) (layer B.Cu) (net 45))
   (segment (start 48.925 49.25) (end 49.75 49.25) (width 0.15) (layer F.Cu) (net 47))
   (segment (start 49.75 49.25) (end 50 49.5) (width 0.15) (layer F.Cu) (net 47))
@@
   (segment (start 40.4 56.4) (end 41.65 56.4) (width 0.15) (layer F.Cu) (net 34))
   (segment (start 41.65 56.4) (end 41.7 56.35) (width 0.15) (layer F.Cu) (net 34))
-  (segment (start 33 46.2) (end 30.6 48.6) (width 0.3) (layer In2.Cu) (net 34))
-  (segment (start 30.6 48.6) (end 30.6 64) (width 0.3) (layer In2.Cu) (net 34))
-  (segment (start 30.6 64) (end 32 65.4) (width 0.3) (layer In2.Cu) (net 34))
-  (segment (start 32 65.4) (end 40.1 65.4) (width 0.3) (layer In2.Cu) (net 34))
-  (segment (start 32.2 29.4) (end 51.3 29.4) (width 0.3) (layer In2.Cu) (net 34))
-  (segment (start 30.6 43.8) (end 30.6 31) (width 0.3) (layer In2.Cu) (net 34))
-  (segment (start 30.6 31) (end 32.2 29.4) (width 0.3) (layer In2.Cu) (net 34))
-  (segment (start 33 46.2) (end 30.6 43.8) (width 0.3) (layer In2.Cu) (net 34))
-  (segment (start 51.3 29.4) (end 52.6 30.7) (width 0.3) (layer In2.Cu) (net 34))
-  (segment (start 52.6 30.7) (end 52.6 32.5) (width 0.3) (layer In2.Cu) (net 34))
-  (segment (start 52.6 32.5) (end 53.63 33.53) (width 0.3) (layer In2.Cu) (net 34))
-  (segment (start 53.63 33.53) (end 55.1 33.53) (width 0.3) (layer In2.Cu) (net 34))
   (segment (start 50 65.4) (end 52.6 65.4) (width 0.3) (layer In2.Cu) (net 34))
   (segment (start 50 64.03) (end 50.02 64.01) (width 0.3) (layer In2.Cu) (net 34))
@@
   (segment (start 50 57.1) (end 50 56.35) (width 0.3) (layer F.Cu) (net 34))
   (via (at 50 57.1) (size 0.5) (drill 0.3) (layers F.Cu B.Cu) (net 34) (status 40000))
-  (segment (start 33 46.2) (end 34.175 46.2) (width 0.3) (layer F.Cu) (net 34))
-  (via (at 33 46.2) (size 0.5) (drill 0.3) (layers F.Cu B.Cu) (net 34))
   (segment (start 43.3 56.15) (end 41.9 56.15) (width 0.3) (layer F.Cu) (net 34))
   (segment (start 41.9 56.15) (end 41.7 56.35) (width 0.3) (layer F.Cu) (net 34))
