File: hardware/bitsy-v0.2a/icebreaker-bitsy.kicad_pcb (KiCad board)
At the start: 4 copper layers, 38.1 x 17.8 mm, 95 parts, among them J1 Conn_01x01, J10 Conn_01x01, J11 Conn_01x01, J12 Conn_01x01, J13 Conn_01x01, J14 Jumper, J15 Jumper, J16 Jumper, J17 Jumper, J18 Jumper, J19 Jumper, J2 Conn_01x01, J20 Conn_01x01, J21 Conn_01x01, J22 Conn_01x01, J23 Conn_01x01, J24 Conn_01x01, J25 Conn_01x01, J26 Conn_01x01, J27 Conn_01x01, J28 Conn_01x01, J29 Conn_01x01, J3 Conn_01x01, J30 Conn_01x01, J31 Conn_01x01, J32 Conn_01x01, J33 Conn_01x01, J34 Conn_01x01, J35 Conn_01x01, J36 Conn_01x01, J37 Conn_01x01, J38 Jumper, J4 Conn_01x01, J41 Conn_01x01, J42 Conn_01x01, J43 Conn_01x01, J44 Conn_01x01, J45 Conn_01x01, J46 Conn_01x01, J47 Conn_01x01, J48 Conn_01x01, J49 Conn_01x01, J5 Conn_01x01, J6 Conn_01x01, J7 Conn_01x01, J8 Conn_01x01, J9 Conn_01x01, P1 USB_OTG, SW1 TACT, U1 USBLC6-2, U2 3.3V, U3 1V2, U5 W25Q, U6 ICE5LP4K-SG48, X1 12MHz

Commit message: Added USB pads for easier debugging and hardwired USB connection.
This patch fixes #8
Parts:
- added P2: UP, pkl_pads:PAD_SMD_1x2.65, B.Cu at (31.6, 43.7)
- added P3: UP, pkl_pads:PAD_SMD_1x2.65, B.Cu at (31.6, 46.2)
- added P4: UP, pkl_pads:PAD_SMD_1x2.65, B.Cu at (31.6, 48.8)
- added P5: UP, pkl_pads:PAD_SMD_1x2.65, B.Cu at (31.6, 51.2)
- moved J38 1.10 mm to (34.0, 44.4), turned to 270 degrees
Routing:
- net +5V: track 29.8 -> 33.5 mm
- net /xUD+: track 1.67 -> 4.74 mm, vias 0 -> 1
- net /xUD-: track 1.65 -> 4.65 mm, vias 0 -> 1
- net GND: track 4.27 -> 6.53 mm
Changed lines of the file:
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@@
-(kicad_pcb (version 20171130) (host pcbnew 5.0.0-rc2-dev-unknown-2da7199~62~ubuntu16.04.1)
+(kicad_pcb (version 20171130) (host pcbnew 5.0.0-rc2-dev-unknown-30a78f0~62~ubuntu16.04.1)
   (general
     (thickness 1.6)
     (drawings 161)
-    (tracks 676)
+    (tracks 696)
     (zones 0)
-    (modules 95)
+    (modules 99)
     (nets 61)
   )
@@
   )
   (setup
-    (last_trace_width 0.15)
+    (last_trace_width 0.3)
     (user_trace_width 0.2)
     (user_trace_width 0.3)
@@
     (mod_text_size 1 1)
     (mod_text_width 0.15)
-    (pad_size 0.95 0.9)
+    (pad_size 2.65 1)
     (pad_drill 0)
     (pad_to_mask_clearance 0.05)
@@
     (add_net "Net-(X1-Pad2)")
   )
+  (module pkl_pads:PAD_SMD_1x2.65 (layer B.Cu)
+    (at 31.637216 51.196445)
+    (fp_text reference P5 (at 0 -2.5) (layer B.Fab) hide
+      (effects (font (size 1 1) (thickness 0.15)) (justify mirror))
+    )
+    (fp_text value UP (at 0 2.2) (layer B.Fab) hide
+      (effects (font (size 1 1) (thickness 0.15)) (justify mirror))
+    )
+    (pad 1 smd roundrect (at 0 0) (size 2.65 1) (layers B.Cu B.Mask)(roundrect_rratio 0.25)
+      (net 7 GND))
+  )
+  (module pkl_pads:PAD_SMD_1x2.65 (layer B.Cu)
+    (at 31.637216 43.69)
+    (fp_text reference P2 (at 0 -2.5) (layer B.Fab) hide
+      (effects (font (size 1 1) (thickness 0.15)) (justify mirror))
+    )
+    (fp_text value UP (at 0 2.2) (layer B.Fab) hide
+      (effects (font (size 1 1) (thickness 0.15)) (justify mirror))
+    )
+    (pad 1 smd roundrect (at 0 0) (size 2.65 1) (layers B.Cu B.Mask)(roundrect_rratio 0.25)
+      (net 10 +5V))
+  )
+  (module pkl_pads:PAD_SMD_1x2.65 (layer B.Cu)
+    (at 31.637216 46.23)
+    (fp_text reference P3 (at 0 -2.5) (layer B.Fab) hide
+      (effects (font (size 1 1) (thickness 0.15)) (justify mirror))
+    )
+    (fp_text value UP (at 0 2.2) (layer B.Fab) hide
+      (effects (font (size 1 1) (thickness 0.15)) (justify mirror))
+    )
+    (pad 1 smd roundrect (at 0 0) (size 2.65 1) (layers B.Cu B.Mask)(roundrect_rratio 0.25)
+      (net 31 /xUD-))
+  )
+  (module pkl_pads:PAD_SMD_1x2.65 (layer B.Cu)
+    (at 31.637216 48.77)
+    (fp_text reference P4 (at 0 -2.5) (layer B.Fab) hide
+      (effects (font (size 1 1) (thickness 0.15)) (justify mirror))
+    )
+    (fp_text value UP (at 0 2.2) (layer B.Fab) hide
+      (effects (font (size 1 1) (thickness 0.15)) (justify mirror))
+    )
+    (pad 1 smd roundrect (at 0 0) (size 2.65 1) (layers B.Cu B.Mask)(roundrect_rratio 0.25)
+      (net 33 /xUD+))
+  )
   (module pkl_jumpers:J_0603 (layer B.Cu)
-    (at 32.9 44.4 90)
+    (at 34 44.4 270)
     (descr "Jumper SMD 0603, reflow soldering")
     (tags "jumper 0603")
     (attr smd)
-    (fp_text reference J38 (at 0 0 90) (layer B.Fab)
+    (fp_text reference J38 (at 0 0 270) (layer B.Fab)
       (effects (font (size 0.635 0.635) (thickness 0.1)) (justify mirror))
     )
-    (fp_text value Jumper (at 0 -1.2 90) (layer B.Fab) hide
+    (fp_text value Jumper (at 0 -1.2 270) (layer B.Fab) hide
       (effects (font (size 0.635 0.635) (thickness 0.1)) (justify mirror))
     )
@@
     (fp_line (start -1.15 0.6) (end 1.15 0.6) (layer B.SilkS) (width 0.13))
     (fp_line (start 1.15 -0.6) (end -1.15 -0.6) (layer B.SilkS) (width 0.13))
-    (pad 1 smd roundrect (at -0.575 0 90) (size 0.95 0.9) (layers B.Cu B.Mask)(roundrect_rratio 0.25)
+    (pad 1 smd roundrect (at -0.575 0 270) (size 0.95 0.9) (layers B.Cu B.Mask)(roundrect_rratio 0.25)
       (net 10 +5V))
-    (pad 2 smd roundrect (at 0.575 0 90) (size 0.95 0.9) (layers B.Cu B.Mask)(roundrect_rratio 0.25)
+    (pad 2 smd roundrect (at 0.575 0 270) (size 0.95 0.9) (layers B.Cu B.Mask)(roundrect_rratio 0.25)
       (net 10 +5V))
   )
@@
     (effects (font (size 0.5 0.5) (thickness 0.125)))
   )
-  (gr_text CC-BY-SA (at 33 49.9 270) (layer B.SilkS)
+  (gr_text CC-BY-SA (at 34 49 270) (layer B.SilkS)
     (effects (font (size 0.75 0.75) (thickness 0.1875)) (justify mirror))
   )
@@
     (effects (font (size 1 1) (thickness 0.25)) (justify mirror))
   )
-  (gr_text VIN (at 34.1 44.4 270) (layer B.SilkS)
+  (gr_text VIN (at 35.3 44.4 270) (layer B.SilkS)
     (effects (font (size 0.75 0.75) (thickness 0.1875)) (justify mirror))
   )
@@
   (segment (start 44.250001 50.250001) (end 44.5 50.5) (width 0.15) (layer F.Cu) (net 6))
   (via (at 44.5 50.5) (size 0.5) (drill 0.3) (layers F.Cu B.Cu) (net 6))
+  (segment (start 34.175 48.8) (end 33.4 48.8) (width 0.3) (layer F.Cu) (net 7))
+  (segment (start 32.7 49.5) (end 32.7 50) (width 0.3) (layer F.Cu) (net 7))
+  (via (at 32.7 50) (size 0.5) (drill 0.3) (layers F.Cu B.Cu) (net 7))
+  (segment (start 33.4 48.8) (end 32.7 49.5) (width 0.3) (layer F.Cu) (net 7))
   (via (at 55.9 42.2) (size 0.5) (drill 0.3) (layers F.Cu B.Cu) (net 7))
   (via (at 36.8 43.49999) (size 0.5) (drill 0.3) (layers F.Cu B.Cu) (net 7))
@@
   (via (at 36.8 42.7) (size 0.5) (drill 0.3) (layers F.Cu B.Cu) (net 7))
   (via (at 30.5 40.8) (size 0.5) (drill 0.3) (layers F.Cu B.Cu) (net 7))
-  (via (at 32.3 41.7) (size 0.5) (drill 0.3) (layers F.Cu B.Cu) (net 7))
   (segment (start 53.978002 42.278002) (end 53.978002 43.074998) (width 0.15) (layer F.Cu) (net 8))
   (segment (start 53.3 41.6) (end 53.978002 42.278002) (width 0.15) (layer F.Cu) (net 8))
@@
   (segment (start 37.9 43.65) (end 37.9 44.5) (width 0.15) (layer F.Cu) (net 9))
   (segment (start 37.9 44.5) (end 38.1 44.7) (width 0.15) (layer F.Cu) (net 9))
+  (segment (start 34.9 42.4) (end 34.4 41.9) (width 0.3) (layer B.Cu) (net 10))
+  (segment (start 34.4 41.9) (end 33.8 41.9) (width 0.3) (layer B.Cu) (net 10))
+  (segment (start 34.9 43.475) (end 34.9 42.4) (width 0.3) (layer B.Cu) (net 10))
+  (segment (start 34 43.825) (end 34.55 43.825) (width 0.3) (layer B.Cu) (net 10))
+  (segment (start 34.55 43.825) (end 34.9 43.475) (width 0.3) (layer B.Cu) (net 10))
+  (segment (start 34 44.975) (end 34 43.825) (width 0.3) (layer B.Cu) (net 10))
+  (segment (start 32.7 45) (end 33.975 45) (width 0.3) (layer B.Cu) (net 10))
+  (segment (start 33.975 45) (end 34 44.975) (width 0.3) (layer B.Cu) (net 10))
+  (segment (start 31.637216 43.69) (end 31.637216 43.937216) (width 0.3) (layer B.Cu) (net 10))
+  (segment (start 31.637216 43.937216) (end 32.7 45) (width 0.3) (layer B.Cu) (net 10))
+  (via (at 32.7 45) (size 0.5) (drill 0.3) (layers F.Cu B.Cu) (net 10))
+  (segment (start 34.175 46.2) (end 33.810034 46.2) (width 0.3) (layer F.Cu) (net 10))
+  (segment (start 32.7 45.089966) (end 32.7 45) (width 0.3) (layer F.Cu) (net 10))
+  (segment (start 33.810034 46.2) (end 32.7 45.089966) (width 0.3) (layer F.Cu) (net 10))
   (segment (start 34.153553 41.9) (end 36.303553 44.05) (width 0.3) (layer In2.Cu) (net 10))
   (segment (start 36.303553 44.05) (end 40.15 44.05) (width 0.3) (layer In2.Cu) (net 10))
@@
   (segment (start 41.010995 41.75) (end 40.7 41.75) (width 0.3) (layer F.Cu) (net 10))
   (segment (start 41.535998 42.275003) (end 41.010995 41.75) (width 0.3) (layer F.Cu) (net 10))
-  (segment (start 32.9 43.825) (end 32.9 42.8) (width 0.3) (layer B.Cu) (net 10))
-  (segment (start 32.9 42.8) (end 33.8 41.9) (width 0.3) (layer B.Cu) (net 10))
-  (segment (start 32.9 44.975) (end 32.9 43.825) (width 0.3) (layer B.Cu) (net 10))
-  (segment (start 33 46.2) (end 33 45.075) (width 0.3) (layer B.Cu) (net 10))
-  (segment (start 33 45.075) (end 32.9 44.975) (width 0.3) (layer B.Cu) (net 10))
-  (segment (start 34.175 46.2) (end 33 46.2) (width 0.3) (layer F.Cu) (net 10))
-  (via (at 33 46.2) (size 0.5) (drill 0.3) (layers F.Cu B.Cu) (net 10))
   (via (at 33.8 41.9) (size 0.5) (drill 0.3) (layers F.Cu B.Cu) (net 10))
   (segment (start 36.1 45.7) (end 36.1 46.25) (width 0.15) (layer F.Cu) (net 10))
@@
   (segment (start 45.250002 46.75) (end 45.200002 46.8) (width 0.15) (layer F.Cu) (net 22))
   (via (at 45.200002 46.8) (size 0.5) (drill 0.3) (layers F.Cu B.Cu) (net 22))
-  (via (at 31.5 50) (size 0.5) (drill 0.3) (layers F.Cu B.Cu) (net 23))
-  (via (at 31.5 45) (size 0.5) (drill 0.3) (layers F.Cu B.Cu) (net 23))
+  (via (at 31.1 50) (size 0.5) (drill 0.3) (layers F.Cu B.Cu) (net 23))
+  (via (at 31.1 45) (size 0.5) (drill 0.3) (layers F.Cu B.Cu) (net 23))
   (via (at 34.1 42.9) (size 0.5) (drill 0.3) (layers F.Cu B.Cu) (net 23))
   (segment (start 31.5 51.3) (end 31.5 52.8) (width 0.15) (layer F.Cu) (net 23))
@@
   (segment (start 39.8 47) (end 40.15 47) (width 0.15) (layer F.Cu) (net 30))
   (segment (start 45.45 47.25) (end 45.9 47.25) (width 0.15) (layer F.Cu) (net 30))
+  (segment (start 33 47.1) (end 32.507216 47.1) (width 0.15) (layer B.Cu) (net 31))
+  (segment (start 32.507216 47.1) (end 31.637216 46.23) (width 0.15) (layer B.Cu) (net 31))
+  (segment (start 34.175 46.85) (end 33.25 46.85) (width 0.15) (layer F.Cu) (net 31))
+  (segment (start 33.25 46.85) (end 33 47.1) (width 0.15) (layer F.Cu) (net 31))
+  (via (at 33 47.1) (size 0.5) (drill 0.3) (layers F.Cu B.Cu) (net 31))
   (segment (start 34.175 46.85) (end 34.95 46.85) (width 0.15) (layer F.Cu) (net 31))
   (segment (start 35.1375 46.6625) (end 35.35 46.6625) (width 0.15) (layer F.Cu) (net 31))
@@
   (segment (start 45.45 47.75) (end 45.9 47.75) (width 0.15) (layer F.Cu) (net 32))
   (segment (start 39.8 48) (end 40.15 48) (width 0.15) (layer F.Cu) (net 32))
+  (segment (start 33 47.9) (end 32.507216 47.9) (width 0.15) (layer B.Cu) (net 33))
+  (segment (start 32.507216 47.9) (end 31.637216 48.77) (width 0.15) (layer B.Cu) (net 33))
+  (segment (start 34.175 47.5) (end 33.4 47.5) (width 0.15) (layer F.Cu) (net 33))
+  (segment (start 33.4 47.5) (end 33 47.9) (width 0.15) (layer F.Cu) (net 33))
+  (via (at 33 47.9) (size 0.5) (drill 0.3) (layers F.Cu B.Cu) (net 33))
   (segment (start 34.175 47.5) (end 34.95 47.5) (width 0.15) (layer F.Cu) (net 33))
   (segment (start 34.95 47.5) (end 35.1875 47.7375) (width 0.15) (layer F.Cu) (net 33))
