File: hardware/v1.0a/icebreaker.kicad_pcb (KiCad board)
At the start: 4 copper layers, 73 x 37 mm, 128 parts, among them J1 Jumper, J10 Jumper, J11 Jumper, J12 Jumper, J13 Jumper, J14 Jumper, J15 Jumper, J16 Jumper, J17 Jumper, J18 Jumper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

Commit message: Add test point for access to FT2232H VREGOUT +1V8 for Powering VCCIO2. See #15 https://github.com/icebreaker-fpga/icebreaker/issues/15
Parts:
- added TP1: TestPoint, TestPoint:TestPoint_Pad_D1.0mm, F.Cu at (50.3, 42.2)
Routing:
- net +1V8: track 32.5 -> 35.2 mm, vias 0 -> 1
