File: hardware/v1.0a/icebreaker.sch (KiCad schematic (older format))
At the start: 121 parts, among them J1 Jumper, J10 Jumper, J11 Jumper, J12 Jumper, J13 Jumper, J14 Jumper, J15 Jumper, J16 Jumper, J17 Jumper, J18 Jumper, J19 Jumper, J2 Jumper, J20 Flash, J21 PMOD_1A, J22 PMOD_1B, J23 PMOD_2H, J24 PMOD_2P, J25 RGB Led, J26 5V AUX, J27 5V AUX, J28 CRESET, J3 Jumper, J4 Jumper, J5 Jumper, J6 Jumper, J7 Jumper, J8 Jumper, J9 Jumper, P1 pkl_USB_OTG, P2 UP, P3 UP, P4 UP, P5 UP, SW1 TACT, SW2 TACT, SW3 TACT, SW4 TACT, U1 93C46B-SOT-23-6, U2 3.3V, U3 1V2, U4 FT2232H, U5 W25Q, U6 ICE5LP4K-SG48, U7 12MHz

Commit message: Add test point for access to FT2232H VREGOUT +1V8 for Powering VCCIO2. See #15 https://github.com/icebreaker-fpga/icebreaker/issues/15
Parts:
- added TP1: TestPoint, TestPoint:TestPoint_Pad_D1.0mm, symbol Connector:TestPoint
Connections:
- wire segments 570 -> 571
Changed lines of the file:
@@
 Text Notes 9800 3800 2    50   ~ 0
 DPair
+$Comp
+L Connector:TestPoint TP1
+U 1 1 5BAE28FE
+P 1550 3450
+F 0 "TP1" H 1608 3570 50  0000 L CNN
+F 1 "TestPoint" H 1608 3479 50  0000 L CNN
+F 2 "TestPoint:TestPoint_Pad_D1.0mm" H 1750 3450 50  0001 C CNN
+F 3 "~" H 1750 3450 50  0001 C CNN
+	1    1550 3450
+	1    0    0    -1
+$EndComp
+Wire Wire Line
+	1550 3450 2100 3450
 $EndSCHEMATC
