File: hardware/v1.0a/icebreaker.sch (KiCad schematic (older format))
At the start: 118 parts, among them J1 Jumper, J10 Jumper, J11 Jumper, J12 Jumper, J13 Jumper, J14 Jumper, J15 Jumper, J16 Jumper, J17 Jumper, J18 Jumper, J19 Jumper, J2 Jumper, J20 Flash, J21 PMOD_1A, J22 PMOD_1B, J23 PMOD_2H, J24 PMOD_2P, J25 RGB Led, J26 5V AUX, J27 5V AUX, J3 Jumper, J4 Jumper, J5 Jumper, J6 Jumper, J7 Jumper, J8 Jumper, J9 Jumper, P1 pkl_USB_OTG, P2 UP, P3 UP, P4 UP, P5 UP, SW1 TACT, SW2 TACT, SW3 TACT, SW4 TACT, U1 93C46B-SOT-23-6, U2 3.3V, U3 1V2, U4 FT2232H, U5 W25Q, U6 ICE5LP4K-SG48, U7 12MHz

Commit message: Use normally closed jumpers. And fix VCCIO2 bypass. Closes #11
These jumpers connect two nets without impacting the schematic net
lists. This is a safer solution and easier to read than having to
remember where the net jumpers have to go and not miss a side path.
These jumpers use a hack of KiCAD where the DRC ignores lines on the
copper layer in footprints. The two pads of the jumper are shorted
within the footprint but they are not from the perspective of the DRC.
While I was already at it I have also replaced / separator with |
separator for multifunction nets. Unfortunately KiCAD reserves the /
separator for its multisheet net naming. This patch should fix the
bypass of the VCCIO0 jumper that was a mistake in the previous versions
of the board.
Parts:
- J1, J15, J16, J18, J2: footprint pkl_jumpers:J_0603 -> pkl_jumpers:J_NC_0603_15; symbol pkl_misc:Jumper -> pkl_misc:pkl_jumper_nc
- J10, J11, J12, J13, J3, J4, J5, J6, J7, J8, J9: symbol pkl_misc:Jumper -> pkl_misc:pkl_jumper
- J14, J17, J19: footprint pkl_jumpers:J_0603 -> pkl_jumpers:J_NC_0603_30; symbol pkl_misc:Jumper -> pkl_misc:pkl_jumper_nc
Connections:
- net labels added: FLASH_CS, VCCIO_0|1, VCCIO_2, VCCPLL, VCORE, xFIFO_D0, xFIFO_D1
- wire segments 612 -> 567

Commit message: Added pulldown on the B port ~CTS ftdi line. Closes #10
With this line pulled down we can use minicom even when hardware flow
control is enabled. If this pin is not pulled low and hardware flow
control is used, no data is ever sent out by the FTDI chip. This can
easily happen because minicom has hardware flow control enabled by
default.

I decided to only add the CTS line pulldown to keep the placements under
control.
Parts:
- added R25: 10k, pkl_dipol:R_0402, symbol pkl_device:pkl_R_Small
Connections:
- wire segments 567 -> 566
Other:
- note added: "RX"
- note added: "TX"
- note added: "TXDEN"
- note added: "~CTS"
- note added: "~DCD"
- note added: "~DSR"
- note added: "~DTR"
- note added: "~RI"
- note added: "~RTS"
- note added: "~RXLED"
- note added: "~TXLED"

Commit message: Mark FTDI flash as optional. Closes #12
Parts:
- C1, R2, R6, U1: DNP (none) -> YES
Other:
- note added: "Optional:\nWe are not programming the\nFTDI flash. We will keep the\nfootprint but will not populate."
Changed lines of the file:
@@
 F 2 "pkl_housings_sot:SOT-23-6" H 1300 5600 50  0001 C CNN
 F 3 "http://ww1.microchip.com/downloads/en/DeviceDoc/20001749K.pdf" H 1300 5950 50  0001 C CNN
-F 4 "EEPROM 1KBit 2MHz SOT-23-6" H 1300 5950 50  0001 C CNN "Description"
-F 5 "93C46B" H 1300 5950 50  0001 C CNN "MFN"
-F 6 "ANY" H 1300 5950 50  0001 C CNN "Source"
-F 7 "eeprom-sot23-6-93c46b" H 0   0   50  0001 C CNN "Key"
+F 4 "eeprom-sot23-6-93c46b" H 0   0   50  0001 C CNN "Key"
+F 5 "EEPROM 1KBit 2MHz SOT-23-6" H 1300 5950 50  0001 C CNN "Description"
+F 6 "93C46B" H 1300 5950 50  0001 C CNN "MFN"
+F 7 "ANY" H 1300 5950 50  0001 C CNN "Source"
+F 8 "YES" H 1300 5950 50  0001 C CNN "DNP"
 	1    1300 5950
 	1    0    0    -1
@@
 F 2 "pkl_dipol:C_0402" H 892 5857 60  0001 L CNN
 F 3 "" H 800 5950 60  0000 C CNN
-F 4 "ANY" H 800 5950 50  0001 C CNN "Source"
-F 5 "cap-cer-0402-100n" H 100 -200 50  0001 C CNN "Key"
+F 4 "cap-cer-0402-100n" H 100 -200 50  0001 C CNN "Key"
+F 5 "ANY" H 800 5950 50  0001 C CNN "Source"
+F 6 "YES" H 800 5950 50  0001 C CNN "DNP"
 	1    800  5950
 	-1   0    0    -1
@@
 F 2 "pkl_dipol:R_0402" H 2259 6057 60  0001 L CNN
 F 3 "" H 2200 6150 60  0000 C CNN
-F 4 "ANY" H 2200 6150 50  0001 C CNN "Source"
-F 5 "res-0402-2k2" H -300 0   50  0001 C CNN "Key"
+F 4 "res-0402-2k2" H -300 0   50  0001 C CNN "Key"
+F 5 "ANY" H 2200 6150 50  0001 C CNN "Source"
+F 6 "YES" H 2200 6150 50  0001 C CNN "DNP"
 	1    2200 6150
 	0    1    1    0
@@
 F 2 "pkl_dipol:R_Array_Convex_4x0402" H 1900 5600 60  0001 C CNN
 F 3 "" H 1900 5600 60  0000 C CNN
-F 4 "ANY" H 1900 5600 50  0001 C CNN "Source"
-F 5 "res-0402cv-array-4-10k" H -100 -50 50  0001 C CNN "Key"
+F 4 "res-0402cv-array-4-10k" H -100 -50 50  0001 C CNN "Key"
+F 5 "ANY" H 1900 5600 50  0001 C CNN "Source"
+F 6 "YES" H 1900 5600 50  0001 C CNN "DNP"
 	1    1900 5600
 	1    0    0    1
@@
 F 2 "pkl_dipol:R_Array_Convex_4x0402" H 1800 5600 60  0001 C CNN
 F 3 "" H 1800 5600 60  0000 C CNN
-F 4 "ANY" H 1800 5600 50  0001 C CNN "Source"
-F 5 "res-0402cv-array-4-10k" H 0   -50 50  0001 C CNN "Key"
+F 4 "res-0402cv-array-4-10k" H 0   -50 50  0001 C CNN "Key"
+F 5 "ANY" H 1800 5600 50  0001 C CNN "Source"
+F 6 "YES" H 1800 5600 50  0001 C CNN "DNP"
 	2    1800 5600
 	1    0    0    1
@@
 F 2 "pkl_dipol:R_Array_Convex_4x0402" H 2000 5600 60  0001 C CNN
 F 3 "" H 2000 5600 60  0000 C CNN
-F 4 "ANY" H 2000 5600 50  0001 C CNN "Source"
-F 5 "res-0402cv-array-4-10k" H -200 -50 50  0001 C CNN "Key"
+F 4 "res-0402cv-array-4-10k" H -200 -50 50  0001 C CNN "Key"
+F 5 "ANY" H 2000 5600 50  0001 C CNN "Source"
+F 6 "YES" H 2000 5600 50  0001 C CNN "DNP"
 	3    2000 5600
 	1    0    0    1
@@
 Wire Wire Line
 	5800 6750 5800 7050
+Text Notes 550  5500 0    50   ~ 0
+Optional:\nWe are not programming the\nFTDI flash. We will keep the\nfootprint but will not populate.
 $EndSCHEMATC

Commit message: Add an FPGA CRESET jumper. Fixes #9
Adding an in line resistor for the CRESET line from FTDI as well as a
jumper that allows access and pulldown of the CRESET line. This allows
us to override the CRESET signal from FTDI and force the FPGA chip to
stay in reset in cases when we need to access the flash and prevent the
FPGA from configuring the FLASH chip. Especially in cases when the FPGA
is using the FLASH after the design is loaded and configures the flash
into QSPI and other higher bit modes.
Parts:
- added J28: CRESET, Connector_PinHeader_2.54mm:PinHeader_2x01_P2.54mm_Vertical, symbol Connector_Generic:Conn_02x01
- added R26: 10k, pkl_dipol:R_0402, symbol pkl_device:pkl_R_Small
Connections:
- net labels added: xiCE_CRESET
- wire segments 566 -> 570
Changed lines of the file:
@@
 	4900 3650 5000 3650
 Wire Wire Line
-	4900 3850 5000 3850
+	4900 3850 6400 3850
 Wire Wire Line
-	4900 3950 5000 3950
+	4900 3950 6000 3950
 NoConn ~ 4900 3550
 NoConn ~ 4900 3750
@@
 Text Label 5000 3650 0    50   ~ 0
 iCE_SS_B
-Text Label 5000 3850 0    50   ~ 0
+Text Label 6400 3850 0    50   ~ 0
 iCE_CDONE
-Text Label 5000 3950 0    50   ~ 0
+Text Label 6400 3950 0    50   ~ 0
 iCE_CRESET
 NoConn ~ 4900 4150
@@
 Text Notes 550  5500 0    50   ~ 0
 Optional:\nWe are not programming the\nFTDI flash. We will keep the\nfootprint but will not populate.
+$Comp
+L pkl_device:pkl_R_Small R26
+U 1 1 5B973233
+P 6100 3950
+F 0 "R26" V 6150 3800 50  0000 C CNN
+F 1 "10k" V 6150 4100 50  0000 C CNN
+F 2 "pkl_dipol:R_0402" H 6159 3857 60  0001 L CNN
+F 3 "" H 6100 3950 60  0000 C CNN
+F 4 "res-0402-10k" H 3600 -2800 50  0001 C CNN "Key"
+F 5 "ANY" H 6100 3950 50  0001 C CNN "Source"
+	1    6100 3950
+	0    1    1    0
+$EndComp
+Wire Wire Line
+	6200 3950 6400 3950
+Text Label 5000 3950 0    50   ~ 0
+xiCE_CRESET
+$Comp
+L Connector_Generic:Conn_02x01 J28
+U 1 1 5BB15B0D
+P 11000 5850
+F 0 "J28" H 11050 6070 50  0000 C CNN
+F 1 "CRESET" H 11050 5977 50  0000 C CNN
+F 2 "Connector_PinHeader_2.54mm:PinHeader_2x01_P2.54mm_Vertical" H 11000 5850 50  0001 C CNN
+F 3 "~" H 11000 5850 50  0001 C CNN
+F 4 "conn-th-01in-2-1-hdr" H -1400 -700 50  0001 C CNN "Key"
+F 5 "ANY" H 11000 5850 50  0001 C CNN "Source"
+	1    11000 5850
+	-1   0    0    1
+$EndComp
+Wire Wire Line
+	11200 5850 11200 5700
+Connection ~ 11200 5700
+Wire Wire Line
+	10700 5850 10600 5850
+Wire Wire Line
+	10600 5850 10600 6100
+$Comp
+L power:GND #PWR0103
+U 1 1 5BBBDFA9
+P 10600 6100
+F 0 "#PWR0103" H 10600 5850 50  0001 C CNN
+F 1 "GND" H 10600 5950 50  0000 C CNN
+F 2 "" H 10600 6100 50  0001 C CNN
+F 3 "" H 10600 6100 50  0001 C CNN
+	1    10600 6100
+	1    0    0    -1
+$EndComp
 $EndSCHEMATC

Commit message: Silkscreen improvements.
Connections:
- net labels added: iCE_SI, iCE_SO
- net labels removed: iCE_MISO, iCE_MOSI
Changed lines of the file:
@@
 iCE_SS_B
 Text Label 8500 4500 2    50   ~ 0
-iCE_MOSI
+iCE_SI
 Text Label 8500 4400 2    50   ~ 0
-iCE_MISO
+iCE_SO
 $Comp
 L pkl_misc:pkl_jumper_nc J18
@@
 L pkl_device:pkl_R4_Small R11
 U 1 1 5AB5AE47
-P 8800 7400
-F 0 "R11" V 8750 7100 50  0000 L CNN
-F 1 "10k" V 8750 7500 50  0000 L CNN
-F 2 "pkl_dipol:R_Array_Convex_4x0402" H 8800 7400 60  0001 C CNN
-F 3 "" H 8800 7400 60  0000 C CNN
-F 4 "ANY" H 8800 7400 50  0001 C CNN "Source"
-F 5 "res-0402cv-array-4-10k" H 0   0   50  0001 C CNN "Key"
-	1    8800 7400
+P 8900 7400
+F 0 "R11" V 8850 7100 50  0000 L CNN
+F 1 "10k" V 8850 7500 50  0000 L CNN
+F 2 "pkl_dipol:R_Array_Convex_4x0402" H 8900 7400 60  0001 C CNN
+F 3 "" H 8900 7400 60  0000 C CNN
+F 4 "ANY" H 8900 7400 50  0001 C CNN "Source"
+F 5 "res-0402cv-array-4-10k" H 100 0   50  0001 C CNN "Key"
+	1    8900 7400
 	1    0    0    -1
 $EndComp
@@
 L pkl_device:pkl_R4_Small R11
 U 4 1 5ABF66A6
-P 8900 7400
-F 0 "R11" V 8850 7100 50  0000 L CNN
-F 1 "10k" V 8850 7500 50  0000 L CNN
-F 2 "pkl_dipol:R_Array_Convex_4x0402" H 8900 7400 60  0001 C CNN
-F 3 "" H 8900 7400 60  0000 C CNN
-F 4 "ANY" H 8900 7400 50  0001 C CNN "Source"
-F 5 "res-0402cv-array-4-10k" H 0   0   50  0001 C CNN "Key"
-	4    8900 7400
+P 8800 7400
+F 0 "R11" V 8750 7100 50  0000 L CNN
+F 1 "10k" V 8750 7500 50  0000 L CNN
+F 2 "pkl_dipol:R_Array_Convex_4x0402" H 8800 7400 60  0001 C CNN
+F 3 "" H 8800 7400 60  0000 C CNN
+F 4 "ANY" H 8800 7400 50  0001 C CNN "Source"
+F 5 "res-0402cv-array-4-10k" H -100 0   50  0001 C CNN "Key"
+	4    8800 7400
 	1    0    0    -1
 $EndComp
@@
 FLASH_MOSI|IO0
 Text Label 7950 8950 2    50   ~ 0
-iCE_MOSI
+iCE_SI
 Text Label 8550 8750 0    50   ~ 0
-iCE_MISO
+iCE_SO
 Text Label 8550 8950 0    50   ~ 0
 FLASH_MISO|IO1

Commit message: Added differential comparator input pin pair groupings.
The symbol in the schematic now shows which pins form diff comparator
input pairs.
Other:
- note added: "DPair"
Changed lines of the file:
@@
 	1    0    0    -1
 $EndComp
+Wire Notes Line
+	9250 2700 9300 2700
+Wire Notes Line
+	9300 2700 9300 2600
+Wire Notes Line
+	9300 2600 9100 2600
+Text Notes 9300 2700 0    50   ~ 0
+DPair
+Wire Notes Line
+	9100 2800 9300 2800
+Wire Notes Line
+	9300 2800 9300 2900
+Wire Notes Line
+	9300 2900 9100 2900
+Text Notes 9300 2900 0    50   ~ 0
+DPair
+Wire Notes Line
+	9100 3100 9300 3100
+Wire Notes Line
+	9300 3100 9300 3200
+Wire Notes Line
+	9300 3200 9100 3200
+Text Notes 9300 3200 0    50   ~ 0
+DPair
+Wire Notes Line
+	10050 4900 9850 4900
+Wire Notes Line
+	9850 4900 9850 5000
+Wire Notes Line
+	9850 5000 10050 5000
+Text Notes 9850 5000 2    50   ~ 0
+DPair
+Wire Notes Line
+	10050 5100 9850 5100
+Wire Notes Line
+	9850 5100 9850 5200
+Wire Notes Line
+	9850 5200 9900 5200
+Text Notes 9850 5200 2    50   ~ 0
+DPair
+Wire Notes Line
+	10050 2500 9850 2500
+Wire Notes Line
+	9850 2500 9850 2600
+Wire Notes Line
+	9850 2600 10050 2600
+Text Notes 9800 2600 2    50   ~ 0
+DPair
+Wire Notes Line
+	10050 2700 9850 2700
+Wire Notes Line
+	9850 2700 9850 2800
+Wire Notes Line
+	9850 2800 10050 2800
+Text Notes 9800 2800 2    50   ~ 0
+DPair
+Wire Notes Line
+	10050 3000 9850 3000
+Wire Notes Line
+	9850 3000 9850 3100
+Wire Notes Line
+	9850 3100 10050 3100
+Text Notes 9800 3100 2    50   ~ 0
+DPair
+Wire Notes Line
+	10050 3200 9850 3200
+Wire Notes Line
+	9850 3200 9850 3300
+Wire Notes Line
+	9850 3300 9900 3300
+Text Notes 9800 3300 2    50   ~ 0
+DPair
+Wire Notes Line
+	10050 3500 9850 3500
+Wire Notes Line
+	9850 3500 9850 3600
+Wire Notes Line
+	9850 3600 10050 3600
+Text Notes 9800 3600 2    50   ~ 0
+DPair
+Wire Notes Line
+	10050 3700 9850 3700
+Wire Notes Line
+	9850 3700 9850 3800
+Wire Notes Line
+	9850 3800 10050 3800
+Text Notes 9800 3800 2    50   ~ 0
+DPair
 $EndSCHEMATC

Commit message: Updated BOM and assembly documentation.
Parts:
- C1, R2, R6, U1: DNP YES -> (none)
- C32, C33, C34, J28: DNP (none) -> YES
- C35: DNP (none) -> YES; Key (none) -> cap-cer-0402-100n
- D2: Key diode-shottky-0603 -> diode-schottky-0603
- D3: value GRN -> BLU; Key led-0603-grn -> led-0603-blu
- J21: value PMOD_1A -> PMOD
- J22: value PMOD_1B -> PMOD
- J23: value PMOD_2H -> PMOD
- J24: value PMOD_2P -> PMOD
- U6: Key ic-ice5lp4k-sg48 -> ic-ice40up5k-sg48
- U7: Key (none) -> xtal-sot23-5-12mhz-osc
Changed lines of the file:
@@
 F 2 "pkl_housings_dfn_qfn:QFN-48-1EP_7x7mm_Pitch0.5mm" H 11900 4400 50  0001 C CNN
 F 3 "" H 11900 4400 50  0001 C CNN
-F 4 "ANY" H 9600 4200 50  0001 C CNN "Source"
-F 5 "ic-ice5lp4k-sg48" H 0   0   50  0001 C CNN "Key"
+F 4 "ic-ice40up5k-sg48" H 0   0   50  0001 C CNN "Key"
+F 5 "ANY" H 9600 4200 50  0001 C CNN "Source"
 	1    9600 4200
 	1    0    0    -1
@@
 F 6 "93C46B" H 1300 5950 50  0001 C CNN "MFN"
 F 7 "ANY" H 1300 5950 50  0001 C CNN "Source"
-F 8 "YES" H 1300 5950 50  0001 C CNN "DNP"
 	1    1300 5950
 	1    0    0    -1
@@
 F 4 "cap-cer-0402-100n" H 100 -200 50  0001 C CNN "Key"
 F 5 "ANY" H 800 5950 50  0001 C CNN "Source"
-F 6 "YES" H 800 5950 50  0001 C CNN "DNP"
 	1    800  5950
 	-1   0    0    -1
@@
 F 4 "res-0402-2k2" H -300 0   50  0001 C CNN "Key"
 F 5 "ANY" H 2200 6150 50  0001 C CNN "Source"
-F 6 "YES" H 2200 6150 50  0001 C CNN "DNP"
 	1    2200 6150
 	0    1    1    0
@@
 F 2 "pkl_dipol:D_0603" V 8150 5800 60  0001 C CNN
 F 3 "" V 8150 5800 60  0000 C CNN
-F 4 "ANY" H 8150 5800 50  0001 C CNN "Source"
-F 5 "diode-shottky-0603" H 0   0   50  0001 C CNN "Key"
+F 4 "diode-schottky-0603" H 0   0   50  0001 C CNN "Key"
+F 5 "ANY" H 8150 5800 50  0001 C CNN "Source"
 	1    8150 5800
 	1    0    0    -1
@@
 P 13700 2400
 F 0 "J21" H 13750 2800 50  0000 C CNN
-F 1 "PMOD_1A" H 13750 2700 50  0000 C CNN
+F 1 "PMOD" H 13750 2700 50  0000 C CNN
 F 2 "Socket_Strips:Socket_Strip_Angled_2x06" H 13700 2400 50  0001 C CNN
 F 3 "~" H 13700 2400 50  0001 C CNN
@@
 P 13700 4100
 F 0 "J22" H 13750 4400 50  0000 C CNN
-F 1 "PMOD_1B" H 13750 3700 50  0000 C CNN
+F 1 "PMOD" H 13750 3700 50  0000 C CNN
 F 2 "Socket_Strips:Socket_Strip_Angled_2x06" H 13700 4100 50  0001 C CNN
 F 3 "~" H 13700 4100 50  0001 C CNN
@@
 P 12700 5600
 F 0 "J23" H 12750 6020 50  0000 C CNN
-F 1 "PMOD_2H" H 12750 5927 50  0000 C CNN
+F 1 "PMOD" H 12750 5927 50  0000 C CNN
 F 2 "Socket_Strips:Socket_Strip_Straight_2x06" H 12700 5600 50  0001 C CNN
 F 3 "~" H 12700 5600 50  0001 C CNN
@@
 P 15000 5500
 F 0 "J24" H 15050 5920 50  0000 C CNN
-F 1 "PMOD_2P" H 15050 5827 50  0000 C CNN
+F 1 "PMOD" H 15050 5827 50  0000 C CNN
 F 2 "Pin_Headers:Pin_Header_Straight_2x06" H 15000 5500 50  0001 C CNN
 F 3 "~" H 15000 5500 50  0001 C CNN
@@
 P 11400 5900
 F 0 "D3" H 11250 6000 50  0000 L CNN
-F 1 "GRN" H 11450 6000 50  0000 L CNN
+F 1 "BLU" H 11450 6000 50  0000 L CNN
 F 2 "pkl_dipol:D_0603" V 11400 5900 60  0001 C CNN
 F 3 "" V 11400 5900 60  0000 C CNN
-F 4 "ANY" H 11400 5900 50  0001 C CNN "Source"
-F 5 "led-0603-grn" H 0   0   50  0001 C CNN "Key"
+F 4 "led-0603-blu" H 0   0   50  0001 C CNN "Key"
+F 5 "ANY" H 11400 5900 50  0001 C CNN "Source"
 	1    11400 5900
 	0    1    1    0
@@
 F 2 "pkl_dipol:C_0603" H 13442 5757 60  0001 L CNN
 F 3 "" H 13350 5850 60  0000 C CNN
-F 4 "ANY" H 13350 5850 50  0001 C CNN "Source"
-F 5 "cap-cer-0603-10u" H 300 0   50  0001 C CNN "Key"
+F 4 "cap-cer-0603-10u" H 300 0   50  0001 C CNN "Key"
+F 5 "ANY" H 13350 5850 50  0001 C CNN "Source"
+F 6 "YES" H 13350 5850 50  0001 C CNN "DNP"
 	1    13350 5850
 	1    0    0    1
@@
 F 2 "pkl_dipol:C_0603" H 14542 4257 60  0001 L CNN
 F 3 "" H 14450 4350 60  0000 C CNN
-F 4 "ANY" H 14450 4350 50  0001 C CNN "Source"
-F 5 "cap-cer-0603-10u" H 1400 0   50  0001 C CNN "Key"
+F 4 "cap-cer-0603-10u" H 1400 0   50  0001 C CNN "Key"
+F 5 "ANY" H 14450 4350 50  0001 C CNN "Source"
+F 6 "YES" H 14450 4350 50  0001 C CNN "DNP"
 	1    14450 4350
 	1    0    0    1
@@
 F 2 "pkl_dipol:C_0603" H 14542 2557 60  0001 L CNN
 F 3 "" H 14450 2650 60  0000 C CNN
-F 4 "ANY" H 14450 2650 50  0001 C CNN "Source"
-F 5 "cap-cer-0603-10u" H 1400 0   50  0001 C CNN "Key"
+F 4 "cap-cer-0603-10u" H 1400 0   50  0001 C CNN "Key"
+F 5 "ANY" H 14450 2650 50  0001 C CNN "Source"
+F 6 "YES" H 14450 2650 50  0001 C CNN "DNP"
 	1    14450 2650
 	1    0    0    1
@@
 F 2 "pkl_dipol:C_0402" H 8442 5907 60  0001 L CNN
 F 3 "" H 8350 6000 60  0000 C CNN
-F 4 "ANY" H 8350 6000 50  0001 C CNN "Source"
+F 4 "cap-cer-0402-100n" H 8350 6000 50  0001 C CNN "Key"
+F 5 "ANY" H 8350 6000 50  0001 C CNN "Source"
+F 6 "YES" H 8350 6000 50  0001 C CNN "DNP"
 	1    8350 6000
 	-1   0    0    -1
@@
 F 4 "res-0402cv-array-4-10k" H -100 -50 50  0001 C CNN "Key"
 F 5 "ANY" H 1900 5600 50  0001 C CNN "Source"
-F 6 "YES" H 1900 5600 50  0001 C CNN "DNP"
 	1    1900 5600
 	1    0    0    1
@@
 F 4 "res-0402cv-array-4-10k" H 0   -50 50  0001 C CNN "Key"
 F 5 "ANY" H 1800 5600 50  0001 C CNN "Source"
-F 6 "YES" H 1800 5600 50  0001 C CNN "DNP"
 	2    1800 5600
 	1    0    0    1
@@
 F 4 "res-0402cv-array-4-10k" H -200 -50 50  0001 C CNN "Key"
 F 5 "ANY" H 2000 5600 50  0001 C CNN "Source"
-F 6 "YES" H 2000 5600 50  0001 C CNN "DNP"
 	3    2000 5600
 	1    0    0    1
@@
 F 2 "pkl_housings_sot:SOT-23-5" H 1500 6700 50  0001 C CNN
 F 3 "" H 1500 6700 50  0001 C CNN
-F 4 "ANY" H 1500 6800 50  0001 C CNN "Source"
+F 4 "xtal-sot23-5-12mhz-osc" H 1500 6800 50  0001 C CNN "Key"
+F 5 "ANY" H 1500 6800 50  0001 C CNN "Source"
 	1    1500 6800
 	-1   0    0    -1
@@
 F 4 "conn-th-01in-2-1-hdr" H -1400 -700 50  0001 C CNN "Key"
 F 5 "ANY" H 11000 5850 50  0001 C CNN "Source"
+F 6 "YES" H 11000 5850 50  0001 C CNN "DNP"
 	1    11000 5850
 	-1   0    0    1

Commit message: Changed the inline CRESET resestor to 2k2.
We need a lower resistor value so that the FTDI chip can reset the FPGA.
Using a 10k resistor results in a voltage divider and the 1.65v is too
high to assert reset.
Parts:
- R26: value 10k -> 2k2; Key res-0402-10k -> res-0402-2k2
Changed lines of the file:
@@
 P 6100 3950
 F 0 "R26" V 6150 3800 50  0000 C CNN
-F 1 "10k" V 6150 4100 50  0000 C CNN
+F 1 "2k2" V 6150 4100 50  0000 C CNN
 F 2 "pkl_dipol:R_0402" H 6159 3857 60  0001 L CNN
 F 3 "" H 6100 3950 60  0000 C CNN
-F 4 "res-0402-10k" H 3600 -2800 50  0001 C CNN "Key"
+F 4 "res-0402-2k2" H 3600 -2800 50  0001 C CNN "Key"
 F 5 "ANY" H 6100 3950 50  0001 C CNN "Source"
 	1    6100 3950
