File: hardware/v1.0b/icebreaker.sch (KiCad schematic (older format))
At the start: 121 parts, among them J1 Jumper, J10 Jumper, J11 Jumper, J12 Jumper, J13 Jumper, J14 Jumper, J15 Jumper, J16 Jumper, J17 Jumper, J18 Jumper, J19 Jumper, J2 Jumper, J20 Flash, J21 PMOD, J22 PMOD, J23 PMOD, J24 PMOD, J25 RGB Led, J26 5V AUX, J27 5V AUX, J28 CRESET, J3 Jumper, J4 Jumper, J5 Jumper, J6 Jumper, J7 Jumper, J8 Jumper, J9 Jumper, P1 pkl_USB_OTG, P2 UP, P3 UP, P4 UP, P5 UP, SW1 TACT, SW2 TACT, SW3 TACT, SW4 TACT, U1 93C46B-SOT-23-6, U2 3.3V, U3 1V2, U4 FT2232H, U5 W25Q, U6 ICE5LP4K-SG48, U7 12MHz

Commit message: Updated tact switch footprints to match the new parts. Closes #17
Parts:
- SW1, SW2, SW3, SW4: footprint pkl_buttons_switches:SW_SPST_KMR2 -> pkl_buttons_switches:SW_SPST_3x4x2.5; Key sw-tact-top-4.2-2.8 -> sw-tact-top-3x4x25
Changed lines of the file:
@@
 F 0 "SW2" H 14850 6650 60  0000 C CNN
 F 1 "TACT" H 14850 6750 60  0000 C CNN
-F 2 "pkl_buttons_switches:SW_SPST_KMR2" H 14600 6575 60  0001 C CNN
+F 2 "pkl_buttons_switches:SW_SPST_3x4x2.5" H 14600 6575 60  0001 C CNN
 F 3 "" H 14600 6575 60  0000 C CNN
-F 4 "sw-tact-top-4.2-2.8" H 0   0   50  0001 C CNN "Key"
+F 4 "sw-tact-top-3x4x25" H 0   0   50  0001 C CNN "Key"
 	1    14600 6600
 	1    0    0    -1
@@
 F 0 "SW3" H 14850 7050 60  0000 C CNN
 F 1 "TACT" H 14850 7150 60  0000 C CNN
-F 2 "pkl_buttons_switches:SW_SPST_KMR2" H 14600 6975 60  0001 C CNN
+F 2 "pkl_buttons_switches:SW_SPST_3x4x2.5" H 14600 6975 60  0001 C CNN
 F 3 "" H 14600 6975 60  0000 C CNN
-F 4 "sw-tact-top-4.2-2.8" H 0   0   50  0001 C CNN "Key"
+F 4 "sw-tact-top-3x4x25" H 0   0   50  0001 C CNN "Key"
 	1    14600 7000
 	1    0    0    -1
@@
 F 0 "SW4" H 14850 7450 60  0000 C CNN
 F 1 "TACT" H 14850 7550 60  0000 C CNN
-F 2 "pkl_buttons_switches:SW_SPST_KMR2" H 14600 7375 60  0001 C CNN
+F 2 "pkl_buttons_switches:SW_SPST_3x4x2.5" H 14600 7375 60  0001 C CNN
 F 3 "" H 14600 7375 60  0000 C CNN
-F 4 "sw-tact-top-4.2-2.8" H 0   0   50  0001 C CNN "Key"
+F 4 "sw-tact-top-3x4x25" H 0   0   50  0001 C CNN "Key"
 	1    14600 7400
 	1    0    0    -1
@@
 F 0 "SW1" H 12800 9800 60  0000 C CNN
 F 1 "TACT" H 13200 9800 60  0000 C CNN
-F 2 "pkl_buttons_switches:SW_SPST_KMR2" H 13000 9625 60  0001 C CNN
+F 2 "pkl_buttons_switches:SW_SPST_3x4x2.5" H 13000 9625 60  0001 C CNN
 F 3 "" H 13000 9625 60  0000 C CNN
-F 4 "sw-tact-top-4.2-2.8" H 0   0   50  0001 C CNN "Key"
+F 4 "sw-tact-top-3x4x25" H 0   0   50  0001 C CNN "Key"
 	1    13000 9650
 	1    0    0    -1
