File: hardware/bitsy-v1.0a/icebreaker-bitsy.sch (KiCad schematic (older format))
At the start: 94 parts, among them J1 3V3, J10 4, J11 1, J12 5, J13 7, J14 6, J15 16, J16 15, J17 18, J18 17, J19 19, J2 3V3, J20 20, J21 21, J22 22, J23 23, J24 8, J25 9, J26 13, J27 14, J28 12, J29 11, J3 VIN, J30 10, J31 CDONE, J32 CRESET, J33 USB_C, J34 PROG, J4 GND, J5 GND, J6 GND, J7 2, J8 3, J9 0, P1 UP, P2 UP, P3 UP, P4 UP, SW1 TACT, U1 USBLC6-2, U2 TLV75512PDRV, U3 TLV75533PDRV, U4 LY68L6400, U5 W25Q, U6 ICE40UP5K-SG48, X1 12MHz

Commit message: Final bitsy-v1.0a
Parts:
- J33: footprint Connector_USB:USB_C_Receptacle_HRO_TYPE-C-31-M-12 -> pkl_connectors:USB_C_Receptacle_HRO_TYPE-C-31-M-12
- JP1, JP5: footprint pkl_jumpers:J_NC_0603_20x2 -> pkl_jumpers:J_NC_0603_40
Changed lines of the file:
@@
 Sheet 1 1
 Title "iCEBreaker-bitsy"
-Date "2020-06-04"
+Date "2020-06-06"
 Rev "v1.0a"
 Comp "1BitSquared"
@@
 F 0 "J33" H 1307 2667 50  0000 C CNN
 F 1 "USB_C" H 1307 2576 50  0000 C CNN
-F 2 "Connector_USB:USB_C_Receptacle_HRO_TYPE-C-31-M-12" H 1350 1800 50  0001 C CNN
+F 2 "pkl_connectors:USB_C_Receptacle_HRO_TYPE-C-31-M-12" H 1350 1800 50  0001 C CNN
 F 3 "https://www.usb.org/sites/default/files/documents/usb_type-c.zip" H 1350 1800 50  0001 C CNN
 	1    1200 1800
@@
 F 0 "JP1" H 2100 900 50  0000 C CNN
 F 1 "Jumper" H 2100 1145 60  0001 C CNN
-F 2 "pkl_jumpers:J_NC_0603_20x2" H 2100 1000 60  0001 C CNN
+F 2 "pkl_jumpers:J_NC_0603_40" H 2100 1000 60  0001 C CNN
 F 3 "" H 2100 1000 60  0000 C CNN
 F 4 "ANY" H 2100 1000 50  0001 C CNN "Source"
@@
 F 0 "JP5" H 6300 3500 50  0000 C CNN
 F 1 "Jumper" H 6300 3745 60  0001 C CNN
-F 2 "pkl_jumpers:J_NC_0603_20x2" H 6300 3600 60  0001 C CNN
+F 2 "pkl_jumpers:J_NC_0603_40" H 6300 3600 60  0001 C CNN
 F 3 "" H 6300 3600 60  0000 C CNN
 F 4 "ANY" H 6300 3600 50  0001 C CNN "Source"

Commit message: WIP pin shuffling
Parts:
- J10: renamed from J11; value 1 -> 3
- J7: renamed from J8; value 3 -> 2
- J8: renamed from J7; value 2 -> 0
- J9: value 0 -> 1
- renumbered J10 to J11, J14 to J13, J13 to J14, J16 to J15, J15 to J16, J19 to J18, J18 to J19, J30 to J26, J29 to J27, J26 to J29, J27 to J30
Connections:
- net FLASH_~HLD~-IO3: now also U6.19 (IOB_29B); no longer U6.13 (IOB_24A)
- net FLASH_~WP~-IO2: now also U6.18 (IOB_31B); no longer U6.12 (IOB_22A)
- net USB_DET: now also U6.37 (IOT_45A_G1); no longer U6.38 (IOT_50B)
- net ~LEDG: now also U6.6 (IOB_13B); no longer U6.37 (IOT_45A_G1)
- net ~LEDR: now also U6.13 (IOB_24A); no longer U6.11 (IOB_20A)
- net ~UBTN: now also U6.36 (IOT_48B); no longer U6.10 (IOB_18A)
- net IOB_0A renamed IOB_0a
- net IOB_0a: now also J7.1 (Pin_1); no longer J8.1 (Pin_1)
- net IOB_13B renamed IOB_13b
- net IOB_13b: now also U6.9 (IOB_16A); no longer U6.6 (IOB_13B)
- net IOB_16A renamed IOB_18a
- net IOB_18a: now also U6.10 (IOB_18A); no longer U6.9 (IOB_16A)
- net IOB_23B renamed IOB_23b
- net IOB_23b: now also J28.1 (Pin_1); no longer J30.1 (Pin_1)
- net IOB_25B_G3 renamed IOB_25b_G3
- net IOB_25b_G3: now also J30.1 (Pin_1); no longer J28.1 (Pin_1)
- net IOB_29B renamed IOB_22a
- net IOB_22a: now also U6.12 (IOB_22A); no longer U6.19 (IOB_29B)
- net IOB_2A renamed IOB_2a
- net IOB_2a: now also J8.1 (Pin_1); no longer J7.1 (Pin_1)
- net IOB_31B renamed IOB_20a
- net IOB_20a: now also U6.11 (IOB_20A); no longer U6.18 (IOB_31B)
- net IOB_3B_G6 renamed IOB_3b_G6
- net IOB_4A renamed IOB_4a
- net IOB_4a: now also J10.1 (Pin_1); no longer J11.1 (Pin_1)
- net IOB_5B renamed IOB_5b
- net IOB_5b: now also J11.1 (Pin_1); no longer J10.1 (Pin_1)
- net IOB_6A renamed IOB_6a
- net IOB_8A renamed IOB_8a
- net IOB_8a: now also J13.1 (Pin_1); no longer J14.1 (Pin_1)
- net IOB_9B renamed IOB_9b
- net IOB_9b: now also J14.1 (Pin_1); no longer J13.1 (Pin_1)
- net IOT_36B renamed IOT_36b
- net IOT_36b: now also J15.1 (Pin_1); no longer J16.1 (Pin_1)
- net IOT_37A renamed IOT_37a
- net IOT_37a: now also J16.1 (Pin_1); no longer J15.1 (Pin_1)
- net IOT_38B renamed IOT_38b
- net IOT_39A renamed IOT_39a
- net IOT_39a: now also J18.1 (Pin_1); no longer J19.1 (Pin_1)
- net IOT_41A renamed IOT_41a
- net IOT_41a: now also J19.1 (Pin_1); no longer J18.1 (Pin_1)
- net IOT_42B renamed IOT_42b
- net IOT_43A renamed IOT_43a
- net IOT_44B renamed IOT_44b
- net IOT_48B renamed IOT_50b
- net IOT_50b: now also U6.38 (IOT_50B); no longer U6.36 (IOT_48B)
- net iCE_SS_B renamed iCE_SS
Other:
- note added: "+"
- note added: "-"
- note added: "DPair"
- moved on the sheet: J10, J11, J13, J14, J15, J16, J18, J19, J23, J24, J25, J26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

Commit message: Final bitsy-v1.0a (for real this time)
Parts:
- removed C7: 100n, pkl_dipol:C_0402, symbol pkl_device:pkl_C_Small
- removed JP5: Jumper, pkl_jumpers:J_NC_0603_40, symbol pkl_misc:pkl_jumper_nc
- removed JP7: Jumper, pkl_jumpers:J_NC_0603_30, symbol pkl_misc:pkl_jumper_nc
- removed R11: 10k, pkl_dipol:R_0402, symbol pkl_device:pkl_R_Small
- renumbered C3 to C1, C20 to C19, C4 to C2, C5 to C3, C1 to C4, C2 to C5, C8 to C6, C6 to C7, C9 to C8, C19 to C9, J8 to J0, J9 to J1, J26 to J10, J27 to J11, J28 to J12, J29 to J13, J30 to J14, J19 to J17, J17 to J18, J18 to J19, J7 to J2, J4 to J24, J5 to J25, J6 to J26, J1 to J27, J2 to J28, J3 to J29, J10 to J3, J31 to J30, J32 to J31, J34 to J32, J11 to J4, J12 to J5, J13 to J6, J14 to J7, J24 to J8, J25 to J9, JP6 to JP5, JP8 to JP6, R12 to R10, R13 to R11, R14 to R12, R15 to R13, R10 to R14, R9 to R8, R8 to R9, U3 to U2, U2 to U3
Connections:
- net VCC is gone; now on net +1V2: C13.1, C14.1, C15.1, C16.1, C17.1, C18.1, R14.2, U6.30 (VCC), U6.5 (VCC)
- net VCCIO_1 is gone; now on net +3V3: C11.1, U6.22 (SPI_VCCIO1)
- net +3V3: no longer R10.2
- net IOB_0a: now also J23.1 (Pin_1); no longer J2.1 (Pin_1)
- net IOB_18a: now also J7.1 (Pin_1); no longer J9.1 (Pin_1)
- net IOB_20a: now also J8.1 (Pin_1); no longer J10.1 (Pin_1)
- net IOB_22a: now also J9.1 (Pin_1); no longer J11.1 (Pin_1)
- net IOB_23b: now also J10.1 (Pin_1); no longer J12.1 (Pin_1)
- net IOB_25b_G3: now also J12.1 (Pin_1); no longer J14.1 (Pin_1)
- net IOB_4a: now also J2.1 (Pin_1); no longer J3.1 (Pin_1)
- net IOB_5b: now also J3.1 (Pin_1); no longer J4.1 (Pin_1)
- net IOB_8a: now also J4.1 (Pin_1); no longer J6.1 (Pin_1)
- net IOB_9b: now also J5.1 (Pin_1); no longer J7.1 (Pin_1)
- net IOT_37a: now also J14.1 (Pin_1); no longer J16.1 (Pin_1)
- net IOT_38b: now also J15.1 (Pin_1); no longer J18.1 (Pin_1)
- net IOT_39a: now also J16.1 (Pin_1); no longer J19.1 (Pin_1)
- net IOT_42b: now also J18.1 (Pin_1); no longer J20.1 (Pin_1)
- net IOT_43a: now also J19.1 (Pin_1); no longer J21.1 (Pin_1)
- net IOT_44b: now also J20.1 (Pin_1); no longer J22.1 (Pin_1)
- net USB_N: now also U6.38 (IOT_50B); no longer U6.42 (IOT_51A)
- net USB_P: now also U6.42 (IOT_51A); no longer U6.43 (IOT_49A)
- net VCCIO_2: now also R10.2
- net ~RGB0: now also D4.1 (RK); no longer D4.2 (BK)
- net ~RGB2: now also D4.2 (BK); no longer D4.1 (RK)
- net FLASH_MISO-IO1 renamed SPI_MISO-IO1
- net FLASH_MOSI-IO0 renamed SPI_MOSI-IO0
- net FLASH_SS renamed FLASH_~CS
- net FLASH_~CS: now also R9.2; no longer R9.4
- net FLASH_~HLD~-IO3 renamed SPI_~HLD~-IO3
- net SPI_~HLD~-IO3: now also J32.10 (Pin_10); no longer J32.9 (Pin_9), R9.2
- net FLASH_~WP~-IO2 renamed SPI_~WP~-IO2
- net SPI_~WP~-IO2: now also J32.9 (Pin_9); no longer J32.10 (Pin_10), R9.8
- net IOB_13b renamed IOB_16a
- net IOB_16a: now also J6.1 (Pin_1); no longer J8.1 (Pin_1)
- net IOB_6a renamed ~BTN
- net ~BTN: now also R10.1, SW1.1; no longer J5.1 (Pin_1)
- net IOT_36b renamed IOT_36b-~LEDR
- net IOT_36b-~LEDR: now also D1.C, J13.1 (Pin_1); no longer J15.1 (Pin_1)
- removed net IOT_50b: J23.1 (Pin_1), U6.38 (IOT_50B)
- net RAM_SS renamed RAM_~CS
- net RAM_~CS: now also R9.6
- net iCE_CDONE renamed CDONE
- net iCE_CRESET renamed ~CRESET
- net ~CRESET: now also R9.8
- net iCE_SCK renamed SPI_SCK
- net SPI_SCK: now also R9.4; no longer R9.6
- net iCE_SS renamed SPI_~CS
- net ~LEDG renamed IOB_13b-~LEDG
- removed net ~LEDR: D1.C, J13.1 (Pin_1), U6.13 (IOB_24A)
- removed net ~UBTN: R10.1, SW1.1, U6.36 (IOT_48B)
- new net IOB_24a: J11.1 (Pin_1), U6.13 (IOB_24A)
- new net IOT_48b: J21.1 (Pin_1), U6.36 (IOT_48B)
- new net IOT_49a: J22.1 (Pin_1), U6.43 (IOT_49A)
Other:
- note added: "Clock"
- note added: "JP3: Remove jumper when only programming iCE\nReplace jumper for programming Flash and for normal operation"
- note added: "Power Pins"
- note added: "QSPI/Programming"
- note removed: "External Clock"
- note removed: "JP2: Remove jumper when only programming iCE\nReplace jumper for programming Flash and for normal operation"
- note removed: "Power\nPins"
- note removed: "Programming"
- moved on the sheet: C1, C2, C3, C4, C5, C6, C7, D1, D2, D3, D4, J10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

Commit message: Regenerate imgs and pdfs
Parts:
- renumbered J33 to J1, J32 to J2, J0 to P0, J1 to P1, J10 to P10, J11 to P11, J12 to P12, J13 to P13, J14 to P14, J15 to P15, J16 to P16, J17 to P17, J18 to P18, J19 to P19, J2 to P2, J20 to P20, J21 to P21, J22 to P22, J23 to P23, J24 to P24, J25 to P25, J26 to P26, J27 to P27, J28 to P28, J29 to P29, J3 to P3, J30 to P30, J31 to P31, P1 to P32, P2 to P33, P3 to P34, P4 to P35, J4 to P4, J5 to P5, J6 to P6, J7 to P7, J8 to P8, J9 to P9
