File: hardware/bitsy-v1.1a/icebreaker-bitsy.kicad_pcb (KiCad board)
At the start: 4 copper layers, 35.6 x 17.8 mm, 94 parts, among them J1 USB_C, J2 PROG, P0 0, P1 1, P10 10, P11 11, P12 12, P13 13, P14 14, P15 15, P16 16, P17 17, P18 18, P19 19, P2 2, P20 20, P21 21, P22 22, P23 23, P24 GND, P25 GND, P26 GND, P27 3V3, P28 3V3, P29 VIN, P3 3, P30 CDONE, P31 CRESET, P32 UP, P33 UP, P34 UP, P35 UP, P4 4, P5 5, P6 6, P7 7, P8 8, P9 9, SW1 TACT, U1 USBLC6-2, U2 TLV75533PDRV, U3 TLV75512PDRV, U4 LY68L6400, U5 W25Q, U6 ICE40UP5K-SG48, X1 12MHz

Commit message: More WIP
Parts:
- removed J2: PROG, pkl_pin_headers:PinHeader_2x05_P2.54mm_Vertical_SMD
- added P36: CS, pkl_pin_headers:Pin_Header_Straight_Round_1x01, F.Cu at (131.8, 94.9)
- added P37: SCK, pkl_pin_headers:Pin_Header_Straight_Round_1x01, F.Cu at (131.8, 97.5)
- added P38: MISO, pkl_pin_headers:Pin_Header_Straight_Round_1x01, F.Cu at (131.8, 100.0)
- added P39: MOSI, pkl_pin_headers:Pin_Header_Straight_Round_1x01, F.Cu at (131.8, 102.5)
- added P40: IO3, pkl_pads:PAD_SMD_R_1x1, B.Cu at (131.8, 105.1)
- added P41: IO2, pkl_pads:PAD_SMD_R_1x1, B.Cu at (134.3, 105.1)
- U5: footprint Package_SO:SOIC-8_5.275x5.275mm_P1.27mm -> Package_SON:WSON-8-1EP_6x5mm_P1.27mm_EP3.4x4.3mm
- moved R13 12.2 mm to (133.4, 104.4), turned to 0 degrees
- moved D3 11.3 mm to (133.4, 105.6), turned to 180 degrees
- moved C7 5.12 mm to (124.7, 94.6), turned to 270 degrees
- moved JP2 3.07 mm to (126.5, 104.5), turned to 180 degrees
- moved R9 2.90 mm to (131.2, 105.0)
- moved U4 1.52 mm to (127.9, 97.3), turned to 90 degrees
- moved JP3 1.50 mm to (126.5, 103.5), turned to 180 degrees
- moved U5 1.41 mm to (126.9, 103.7)
- moved C11 0.56 mm to (124.7, 98.8), turned to 270 degrees
- moved C8 0.18 mm to (124.7, 96.7), turned to 90 degrees
Connections:
- net /SPI_PISO-IO1 renamed /SPI_MISO-IO1
- net /SPI_POSI-IO0 renamed /SPI_MOSI-IO0
- R9 pad 2: /FLASH_~CS -> /SPI_SCK
- R9 pad 4: /SPI_SCK -> /~CRESET
- R9 pad 6: /RAM_~CS -> /FLASH_~CS
- R9 pad 8: /~CRESET -> /RAM_~CS
Routing:
- net /CDONE: track 25.3 -> 2.19 mm, vias 2 -> 1
- net /~CRESET: track 29.0 -> 13.7 mm
- net /FLASH_~CS: track 9.58 -> 1.45 mm, vias 1 -> 0
- net +3V3: track 30.1 -> 22.5 mm, vias 10 -> 9
- net /SPI_SCK: track 22.5 -> 16.5 mm, vias 2 -> 3
- net /RAM_~CS: track 20.0 -> 14.5 mm, vias 1 -> 0
- net /IOB_25b_G3: track 18.1 -> 23.0 mm
- net /SPI_~CS: track 11.8 -> 16.4 mm
- net /SPI_MOSI-IO0: track 21.5 -> 25.4 mm, vias 3 -> 1
- net GND: track 45.7 -> 42.1 mm
- net /IOB_23b: track 13.5 -> 17.0 mm
- net /SPI_~HLD~-IO3: track 21.1 -> 24.4 mm, vias 2 -> 4
- net /SPI_~WP~-IO2: track 21.6 -> 24.0 mm, vias 2 -> 1
- net /IOB_13b-~LEDG: track 28.7 -> 26.7 mm
- net /SPI_MISO-IO1: track 17.9 -> 16.2 mm, vias 2 -> 0
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Other:
- outline, holes or cut-outs redrawn
- board text added: "B"
- board text added: "D+"
- board text added: "D-"
- board text added: "Flash"
- board text added: "MISO/IO1"
- board text added: "MOSI/IO0"
- board text added: "RAM"
- board text added: "~CS"
- board text removed: "+D"
- board text removed: "-D"
- board text removed: "/"
- board text removed: "BUTTON"
- board text removed: "CDON"
- board text removed: "CRST"
- board text removed: "F"
- board text removed: "FLASH"
- board text removed: "PSRAM"
- board text removed: "QSPI Prog"

Commit message: More WIP
Parts:
- turned SW1 to 0 degrees
Connections:
- SW1 pad 1: /~BTN -> GND
- SW1 pad 2: GND -> /~BTN

Commit message: More routing
Routing:
- net /CDONE: track 2.19 -> 23.4 mm
- net /~CRESET: track 13.7 -> 34.9 mm, vias 1 -> 2
- net /SPI_SCK: track 16.5 -> 28.0 mm
- net /RAM_~CS: track 14.5 -> 15.7 mm

Commit message: Finish up v1.1a
Still TODO:
- check LED resistor values, sync to PCB file
- check JP3 comment in schematic
- should P36 be connected to SPI_CS or FLASH_CS?
- update ibom.html
- update PDFs
- finish top/bottom info sheets
- update README
Parts:
- moved JP3 2.12 mm to (125.0, 102.0), turned to 270 degrees
- moved JP2 1.50 mm to (125.0, 104.5), turned to 270 degrees
- moved R13 0.50 mm to (133.7, 104.0)
- moved REF** 0.10 mm to (122.3, 104.9)
Connections:
- R9 pad 4: /~CRESET -> /FLASH_~CS
- R9 pad 5: +3V3 -> /~CRESET
- R9 pad 6: /FLASH_~CS -> +3V3
- R9 pad 7: +3V3 -> /RAM_~CS
- R9 pad 8: /RAM_~CS -> +3V3
Routing:
- net /CDONE: track 23.4 -> 33.8 mm
- net /RAM_~CS: track 15.7 -> 23.4 mm, vias 0 -> 1
- net /FLASH_~CS: track 1.45 -> 9.13 mm, vias 0 -> 1
- net /~CRESET: track 34.9 -> 28.8 mm
- net +3V3: track 22.5 -> 28.3 mm
- net /IOB_23b: track 17.0 -> 19.9 mm
- net /SPI_~CS: track 16.4 -> 13.6 mm, vias 1 -> 2
- net GND: track 42.1 -> 43.7 mm, vias 13 -> 14
- net /IOB_13b-~LEDG: track 26.7 -> 25.4 mm
- net /IOB_0a: track 17.0 -> 18.0 mm
- net /SPI_~WP~-IO2: track 24.0 -> 24.8 mm
- net /SPI_~HLD~-IO3: track 24.4 -> 25.3 mm
Other:
- board text added: "BTN"
- board text added: "Bitsy"
- board text added: "Flash CS"
- board text added: "IO0"
- board text added: "IO1"
- board text added: "LEDG"
- board text added: "LEDR"
- board text added: "RAM CS"
- board text added: "iCEBitsy v1.1a"
- board text added: "~CRESET"
- board text removed: "B"
- board text removed: "Flash"
- board text removed: "MISO/IO1"
- board text removed: "MOSI/IO0"
- board text removed: "PISO"
- board text removed: "POSI"
- board text removed: "R"
- board text removed: "RAM"
- board text removed: "bitsy"
- board text removed: "iCEBreaker bitsy"

Commit message: Finish up some more TODOs
- change LED resistor values
- update interactive BOM
- update PDFs
- clean up PCB planes & comments
Parts:
- R11, R12: value 330E -> 2k2
- U5: value W25Q -> W25Q128JVxxM
