File: hardware/bitsy-v1.1a/icebreaker-bitsy.sch (KiCad schematic (older format))
At the start: 90 parts, among them J1 USB_C, J2 PROG, P0 0, P1 1, P10 10, P11 11, P12 12, P13 13, P14 14, P15 15, P16 16, P17 17, P18 18, P19 19, P2 2, P20 20, P21 21, P22 22, P23 23, P24 GND, P25 GND, P26 GND, P27 3V3, P28 3V3, P29 VIN, P3 3, P30 CDONE, P31 CRESET, P32 UP, P33 UP, P34 UP, P35 UP, P4 4, P5 5, P6 6, P7 7, P8 8, P9 9, SW1 TACT, U1 USBLC6-2, U2 TLV75533PDRV, U3 TLV75512PDRV, U4 LY68L6400, U5 W25Q, U6 ICE40UP5K-SG48, X1 12MHz

Commit message: More WIP
Parts:
- removed J2: PROG, pkl_pin_headers:PinHeader_2x05_P2.54mm_Vertical_SMD, symbol Connector_Generic:Conn_02x05_Odd_Even
- added P36: CS, pkl_pin_headers:Pin_Header_Straight_Round_1x01, symbol Connector_Generic:Conn_01x01
- added P37: SCK, pkl_pin_headers:Pin_Header_Straight_Round_1x01, symbol Connector_Generic:Conn_01x01
- added P38: MISO, pkl_pin_headers:Pin_Header_Straight_Round_1x01, symbol Connector_Generic:Conn_01x01
- added P39: MOSI, pkl_pin_headers:Pin_Header_Straight_Round_1x01, symbol Connector_Generic:Conn_01x01
- added P40: IO3, pkl_pads:PAD_SMD_R_1x1, symbol Connector_Generic:Conn_01x01
- added P41: IO2, pkl_pads:PAD_SMD_R_1x1, symbol Connector_Generic:Conn_01x01
Connections:
- net FLASH_~CS: now also R9.6; no longer R9.2
- net RAM_~CS: now also R9.8; no longer R9.6
- net SPI_SCK: now also R9.2, P37.1 (Pin_1); no longer R9.4
- net SPI_~CS: now also P36.1 (Pin_1)
- net SPI_~HLD~-IO3: now also P40.1 (Pin_1)
- net SPI_~WP~-IO2: now also P41.1 (Pin_1)
- net ~CRESET: now also R9.4; no longer R9.8
- net SPI_PISO-IO1 renamed SPI_MISO-IO1
- net SPI_MISO-IO1: now also P38.1 (Pin_1)
- net SPI_POSI-IO0 renamed SPI_MOSI-IO0
- net SPI_MOSI-IO0: now also P39.1 (Pin_1)
Other:
- note added: "128M\nFlash"
- note added: "64M\nPSRAM"
- moved on the sheet: R9A, R9B, R9C, R9D
Changed lines of the file:
@@
 Title "iCEBreaker-bitsy"
 Date "2020-06-10"
-Rev "v1.0a"
+Rev "v1.1a"
 Comp "1BitSquared"
 Comment1 "© 2018-2020 1BitSquared <info@1bitsquared.com>"
@@
 SPI_SCK
 Text Label 7500 3400 2    50   ~ 0
-SPI_PISO-IO1
+SPI_MISO-IO1
 Text Label 7500 3300 2    50   ~ 0
-SPI_POSI-IO0
+SPI_MOSI-IO0
 Text Label 5200 3500 0    50   ~ 0
 CDONE
@@
 	3900 2500 3900 2600
 Wire Wire Line
-	9600 4600 10300 4600
+	9600 4600 10200 4600
 $Comp
 L pkl_device:pkl_C_Small C9
@@
 Wire Notes Line
 	4600 7700 4600 6500
-Wire Wire Line
-	6000 7200 6550 7200
-Wire Wire Line
-	6000 7100 6100 7100
-$Comp
-L power:+3.3V #PWR0111
-U 1 1 5EF49BD0
-P 6000 7400
-F 0 "#PWR0111" H 6000 7250 50  0001 C CNN
-F 1 "+3.3V" V 6015 7528 50  0000 L CNN
-F 2 "" H 6000 7400 50  0001 C CNN
-F 3 "" H 6000 7400 50  0001 C CNN
-	1    6000 7400
-	0    1    -1   0
-$EndComp
-Text Label 6100 7200 0    50   ~ 0
-~CRESET
-Text Label 6100 7100 0    50   ~ 0
-CDONE
-Text Label 5400 7100 2    50   ~ 0
-SPI_~CS
-Text Label 5400 7200 2    50   ~ 0
-SPI_SCK
-Text Label 5400 7300 2    50   ~ 0
-SPI_PISO-IO1
-Text Label 5400 7400 2    50   ~ 0
-SPI_POSI-IO0
-Text Label 6100 7500 0    50   ~ 0
-SPI_~WP~-IO2
-Text Label 5400 7500 2    50   ~ 0
-SPI_~HLD~-IO3
-$Comp
-L Connector_Generic:Conn_02x05_Odd_Even J2
-U 1 1 5EF51AE9
-P 5800 7300
-F 0 "J2" H 5850 7717 50  0000 C CNN
-F 1 "PROG" H 5850 7626 50  0000 C CNN
-F 2 "pkl_pin_headers:PinHeader_2x05_P2.54mm_Vertical_SMD" H 5800 7300 50  0001 C CNN
-F 3 "~" H 5800 7300 50  0001 C CNN
-	1    5800 7300
-	-1   0    0    -1
-$EndComp
-Wire Wire Line
-	5500 7100 5400 7100
-Wire Wire Line
-	5500 7200 5400 7200
-$Comp
-L power:GND #PWR0120
-U 1 1 5EFA44D2
-P 6000 7300
-F 0 "#PWR0120" H 6000 7050 50  0001 C CNN
-F 1 "GND" V 6005 7172 50  0000 R CNN
-F 2 "" H 6000 7300 50  0001 C CNN
-F 3 "" H 6000 7300 50  0001 C CNN
-	1    6000 7300
-	0    -1   -1   0
-$EndComp
-Wire Wire Line
-	5500 7500 5400 7500
-Wire Wire Line
-	5400 7300 5500 7300
-Wire Wire Line
-	5400 7400 5500 7400
-Wire Wire Line
-	6000 7500 6100 7500
-Wire Wire Line
-	6550 7200 6550 7000
-$Comp
-L power:+3V3 #PWR0121
-U 1 1 5F121167
-P 6550 6800
-F 0 "#PWR0121" H 6550 6650 50  0001 C CNN
-F 1 "+3V3" H 6550 6950 50  0000 C CNN
-F 2 "" H 6550 6800 50  0001 C CNN
-F 3 "" H 6550 6800 50  0001 C CNN
-	1    6550 6800
-	1    0    0    -1
-$EndComp
-$Comp
-L pkl_device:pkl_R4_Small R9
-U 4 1 5ABF66A6
-P 6550 6900
-F 0 "R9" V 6500 6650 50  0000 L CNN
-F 1 "10k" V 6600 6650 50  0000 L CNN
-F 2 "pkl_dipol:R_Array_Convex_4x0402" H 6550 6900 60  0001 C CNN
-F 3 "" H 6550 6900 60  0000 C CNN
-F 4 "ANY" H 6550 6900 50  0001 C CNN "Source"
-F 5 "res-0402cv-array-4-10k" H -2350 -500 50  0001 C CNN "Key"
-	4    6550 6900
-	1    0    0    -1
-$EndComp
 Wire Notes Line
 	6000 4800 4600 4800
@@
 	2900 5500 2900 5300
 Wire Wire Line
-	2800 5300 2800 5500
-Wire Wire Line
 	2900 5300 2800 5300
 $Comp
-L power:+3V3 #PWR?
+L power:+3V3 #PWR0125
 U 1 1 5F107E69
 P 2900 5300
-F 0 "#PWR?" H 2900 5150 50  0001 C CNN
+F 0 "#PWR0125" H 2900 5150 50  0001 C CNN
 F 1 "+3V3" H 2900 5450 50  0000 C CNN
 F 2 "" H 2900 5300 50  0001 C CNN
@@
 $Comp
 L pkl_device:pkl_R4_Small R9
-U 3 1 5ABF6624
-P 2800 5600
-F 0 "R9" V 2750 5350 50  0000 L CNN
-F 1 "10k" V 2750 5700 50  0000 L CNN
-F 2 "pkl_dipol:R_Array_Convex_4x0402" H 2800 5600 60  0001 C CNN
-F 3 "" H 2800 5600 60  0000 C CNN
-F 4 "ANY" H 2800 5600 50  0001 C CNN "Source"
-F 5 "res-0402cv-array-4-10k" H -5800 -1800 50  0001 C CNN "Key"
-	3    2800 5600
+U 2 1 5AB5B376
+P 10900 4500
+F 0 "R9" V 10850 4250 50  0000 L CNN
+F 1 "10k" V 10950 4250 50  0000 L CNN
+F 2 "pkl_dipol:R_Array_Convex_4x0402" H 10900 4500 60  0001 C CNN
+F 3 "" H 10900 4500 60  0000 C CNN
+F 4 "ANY" H 10900 4500 50  0001 C CNN "Source"
+F 5 "res-0402cv-array-4-10k" H 2200 -2900 50  0001 C CNN "Key"
+	2    10900 4500
 	1    0    0    -1
 $EndComp
 $Comp
 L pkl_device:pkl_R4_Small R9
-U 2 1 5AB5B376
+U 1 1 5AB5AE47
 P 2900 5600
 F 0 "R9" V 2850 5350 50  0000 L CNN
@@
 F 3 "" H 2900 5600 60  0000 C CNN
 F 4 "ANY" H 2900 5600 50  0001 C CNN "Source"
-F 5 "res-0402cv-array-4-10k" H -5800 -1800 50  0001 C CNN "Key"
-	2    2900 5600
-	1    0    0    -1
-$EndComp
-$Comp
-L pkl_device:pkl_R4_Small R9
-U 1 1 5AB5AE47
-P 3000 5600
-F 0 "R9" V 2950 5350 50  0000 L CNN
-F 1 "10k" V 2950 5700 50  0000 L CNN
-F 2 "pkl_dipol:R_Array_Convex_4x0402" H 3000 5600 60  0001 C CNN
-F 3 "" H 3000 5600 60  0000 C CNN
-F 4 "ANY" H 3000 5600 50  0001 C CNN "Source"
-F 5 "res-0402cv-array-4-10k" H -5800 -1800 50  0001 C CNN "Key"
-	1    3000 5600
+F 5 "res-0402cv-array-4-10k" H -5900 -1800 50  0001 C CNN "Key"
+	1    2900 5600
 	1    0    0    -1
 $EndComp
@@
 SPI_SCK
 Text Label 3100 7000 0    50   ~ 0
-SPI_POSI-IO0
+SPI_MOSI-IO0
 Text Label 3100 7100 0    50   ~ 0
-SPI_PISO-IO1
+SPI_MISO-IO1
 Text Label 3100 7200 0    50   ~ 0
 SPI_~WP~-IO2
@@
 	6000 4800 6000 6400
 $Comp
-L power:GND #PWR?
+L power:GND #PWR0126
 U 1 1 5F68FCC7
 P 6900 6100
-F 0 "#PWR?" H 6900 5850 50  0001 C CNN
+F 0 "#PWR0126" H 6900 5850 50  0001 C CNN
 F 1 "GND" H 6900 5950 50  0000 C CNN
 F 2 "" H 6900 6100 50  0001 C CNN
@@
 $EndComp
 $Comp
-L power:GND #PWR?
+L power:GND #PWR0127
 U 1 1 5F68FA7B
 P 6600 6100
-F 0 "#PWR?" H 6600 5850 50  0001 C CNN
+F 0 "#PWR0127" H 6600 5850 50  0001 C CNN
 F 1 "GND" H 6600 5950 50  0000 C CNN
 F 2 "" H 6600 6100 50  0001 C CNN
@@
 $EndComp
 $Comp
-L power:+3V3 #PWR?
+L power:+3V3 #PWR0128
 U 1 1 5F6139CB
 P 7500 5800
-F 0 "#PWR?" H 7500 5650 50  0001 C CNN
+F 0 "#PWR0128" H 7500 5650 50  0001 C CNN
 F 1 "+3V3" H 7500 5950 50  0000 C CNN
 F 2 "" H 7500 5800 50  0001 C CNN
@@
 	0    -1   -1   0
 $EndComp
+$Comp
+L power:+3V3 #PWR0121
+U 1 1 5F121167
+P 10900 4400
+F 0 "#PWR0121" H 10900 4250 50  0001 C CNN
+F 1 "+3V3" H 10900 4550 50  0000 C CNN
+F 2 "" H 10900 4400 50  0001 C CNN
+F 3 "" H 10900 4400 50  0001 C CNN
+	1    10900 4400
+	1    0    0    -1
+$EndComp
+Text Notes 1500 6250 0    50   ~ 0
+64M\nPSRAM
+Text Notes 1500 7150 0    50   ~ 0
+128M\nFlash
+Wire Wire Line
+	2800 5300 2800 5500
+$Comp
+L pkl_device:pkl_R4_Small R9
+U 4 1 5ABF66A6
+P 2800 5600
+F 0 "R9" V 2750 5350 50  0000 L CNN
+F 1 "10k" V 2750 5700 50  0000 L CNN
+F 2 "pkl_dipol:R_Array_Convex_4x0402" H 2800 5600 60  0001 C CNN
+F 3 "" H 2800 5600 60  0000 C CNN
+F 4 "ANY" H 2800 5600 50  0001 C CNN "Source"
+F 5 "res-0402cv-array-4-10k" H -6100 -1800 50  0001 C CNN "Key"
+	4    2800 5600
+	1    0    0    -1
+$EndComp
+$Comp
+L pkl_device:pkl_R4_Small R9
+U 3 1 5ABF6624
+P 3000 5600
+F 0 "R9" V 2950 5350 50  0000 L CNN
+F 1 "10k" V 2950 5700 50  0000 L CNN
+F 2 "pkl_dipol:R_Array_Convex_4x0402" H 3000 5600 60  0001 C CNN
+F 3 "" H 3000 5600 60  0000 C CNN
+F 4 "ANY" H 3000 5600 50  0001 C CNN "Source"
+F 5 "res-0402cv-array-4-10k" H -5600 -1800 50  0001 C CNN "Key"
+	3    3000 5600
+	1    0    0    -1
+$EndComp
+Wire Wire Line
+	10200 4600 10200 4800
+Wire Wire Line
+	10200 4800 10900 4800
+Wire Wire Line
+	10900 4800 10900 4600
+Connection ~ 10200 4600
+Wire Wire Line
+	10200 4600 10300 4600
+$Comp
+L Connector_Generic:Conn_01x01 P41
+U 1 1 5F35ED22
+P 5500 7500
+F 0 "P41" H 5580 7496 50  0000 L CNN
+F 1 "IO2" H 5580 7451 50  0001 L CNN
+F 2 "pkl_pads:PAD_SMD_R_1x1" H 5500 7500 50  0001 C CNN
+F 3 "~" H 5500 7500 50  0001 C CNN
+	1    5500 7500
+	-1   0    0    -1
+$EndComp
+Text Label 5800 7000 0    50   ~ 0
+SPI_~CS
+Text Label 5800 7100 0    50   ~ 0
+SPI_SCK
+Text Label 5800 7200 0    50   ~ 0
+SPI_MISO-IO1
+Text Label 5800 7300 0    50   ~ 0
+SPI_MOSI-IO0
+Text Label 5800 7400 0    50   ~ 0
+SPI_~HLD~-IO3
+Wire Wire Line
+	5700 7000 5800 7000
+Wire Wire Line
+	5700 7100 5800 7100
+Wire Wire Line
+	5700 7400 5800 7400
+Wire Wire Line
+	5800 7200 5700 7200
+Wire Wire Line
+	5800 7300 5700 7300
+$Comp
+L Connector_Generic:Conn_01x01 P36
+U 1 1 5F31319B
+P 5500 7000
+F 0 "P36" H 5580 6996 50  0000 L CNN
+F 1 "CS" H 5580 6951 50  0001 L CNN
+F 2 "pkl_pin_headers:Pin_Header_Straight_Round_1x01" H 5500 7000 50  0001 C CNN
+F 3 "~" H 5500 7000 50  0001 C CNN
+	1    5500 7000
+	-1   0    0    -1
+$EndComp
+$Comp
+L Connector_Generic:Conn_01x01 P37
+U 1 1 5F31B068
+P 5500 7100
+F 0 "P37" H 5580 7096 50  0000 L CNN
+F 1 "SCK" H 5580 7051 50  0001 L CNN
+F 2 "pkl_pin_headers:Pin_Header_Straight_Round_1x01" H 5500 7100 50  0001 C CNN
+F 3 "~" H 5500 7100 50  0001 C CNN
+	1    5500 7100
+	-1   0    0    -1
+$EndComp
+$Comp
+L Connector_Generic:Conn_01x01 P38
+U 1 1 5F31B224
+P 5500 7200
+F 0 "P38" H 5580 7196 50  0000 L CNN
+F 1 "MISO" H 5580 7151 50  0001 L CNN
+F 2 "pkl_pin_headers:Pin_Header_Straight_Round_1x01" H 5500 7200 50  0001 C CNN
+F 3 "~" H 5500 7200 50  0001 C CNN
+	1    5500 7200
+	-1   0    0    -1
+$EndComp
+$Comp
+L Connector_Generic:Conn_01x01 P39
+U 1 1 5F31B48D
+P 5500 7300
+F 0 "P39" H 5580 7296 50  0000 L CNN
+F 1 "MOSI" H 5580 7251 50  0001 L CNN
+F 2 "pkl_pin_headers:Pin_Header_Straight_Round_1x01" H 5500 7300 50  0001 C CNN
+F 3 "~" H 5500 7300 50  0001 C CNN
+	1    5500 7300
+	-1   0    0    -1
+$EndComp
+$Comp
+L Connector_Generic:Conn_01x01 P40
+U 1 1 5F31CDE3
+P 5500 7400
+F 0 "P40" H 5580 7396 50  0000 L CNN
+F 1 "IO3" H 5580 7351 50  0001 L CNN
+F 2 "pkl_pads:PAD_SMD_R_1x1" H 5500 7400 50  0001 C CNN
+F 3 "~" H 5500 7400 50  0001 C CNN
+	1    5500 7400
+	-1   0    0    -1
+$EndComp
+Text Label 5800 7500 0    50   ~ 0
+SPI_~WP~-IO2
+Wire Wire Line
+	5800 7500 5700 7500
 $EndSCHEMATC

Commit message: More WIP
Connections:
- net GND: now also SW1.1; no longer SW1.2
- net ~BTN: now also SW1.2; no longer SW1.1
Changed lines of the file:
@@
 F 4 "sw-tact-top-4.2-2.8" H -9400 -6750 50  0001 C CNN "Key"
 	1    3600 2900
-	-1   0    0    -1
+	1    0    0    -1
 $EndComp
 Wire Wire Line

Commit message: More routing
Other:
- note added: "SPI Terminology:\nMOSI - Main Out Secondary In\nMISO - Main In Secondary Out\nSCK - Serial Clock\nCS - Chip Select"
Changed lines of the file:
@@
 Wire Wire Line
 	5800 7500 5700 7500
+Text Notes 6300 3150 0    50   ~ 0
+SPI Terminology:\nMOSI - Main Out Secondary In\nMISO - Main In Secondary Out\nSCK  - Serial Clock\nCS   - Chip Select
 $EndSCHEMATC

Commit message: Finish up v1.1a
Still TODO:
- check LED resistor values, sync to PCB file
- check JP3 comment in schematic
- should P36 be connected to SPI_CS or FLASH_CS?
- update ibom.html
- update PDFs
- finish top/bottom info sheets
- update README
Parts:
- R11, R12: value 330E -> 2k2
- U5: value W25Q -> W25Q128JVxxM
Connections:
- net +3V3: now also R9.6, R9.8; no longer R9.5, R9.7
- net FLASH_~CS: now also R9.4; no longer R9.6
- net RAM_~CS: now also R9.7; no longer R9.8
- net ~CRESET: now also R9.5; no longer R9.4
Other:
- note added: "Chip Select"
- note added: "Hold"
- note added: "JP3: Cut jumper when only programming iCE\nConnect jumper for programming Flash and for normal operation"
- note added: "Main In Secondary Out"
- note added: "Main Out Secondary In"
- note added: "Serial Clock"
- note added: "Write Protect"
- note removed: "JP3: Remove jumper when only programming iCE\nReplace jumper for programming Flash and for normal operation"
- note removed: "SPI Terminology:\nMOSI - Main Out Secondary In\nMISO - Main In Secondary Out\nSCK - Serial Clock\nCS - Chip Select"
- moved on the sheet: P36, P37, P38, P39, P40, P41, R9B, R9C
Changed lines of the file:
@@
 Sheet 1 1
 Title "iCEBreaker-bitsy"
-Date "2020-06-10"
+Date "2020-08-04"
 Rev "v1.1a"
 Comp "1BitSquared"
@@
 P 5600 2700
 F 0 "R11" V 5700 2700 50  0000 C CNN
-F 1 "330E" V 5500 2700 50  0000 C CNN
+F 1 "2k2" V 5500 2700 50  0000 C CNN
 F 2 "pkl_dipol:R_0402" H 5659 2607 60  0001 L CNN
 F 3 "" H 5600 2700 60  0000 C CNN
@@
 P 5600 3100
 F 0 "R12" V 5700 3100 50  0000 C CNN
-F 1 "330E" V 5500 3100 50  0000 C CNN
+F 1 "2k2" V 5500 3100 50  0000 C CNN
 F 2 "pkl_dipol:R_0402" H 5659 3007 60  0001 L CNN
 F 3 "" H 5600 3100 60  0000 C CNN
@@
 Wire Wire Line
 	5800 4200 5800 3500
-$Comp
-L pkl_memory:W25Q U5
-U 1 1 5A9D24AF
-P 1800 7000
-F 0 "U5" H 1800 7400 50  0000 C CNN
-F 1 "W25Q" H 1800 7300 50  0000 C CNN
-F 2 "Package_SON:WSON-8-1EP_6x5mm_P1.27mm_EP3.4x4.3mm" H 1800 7000 50  0001 C CNN
-F 3 "" H 1800 7000 50  0001 C CNN
-F 4 "ANY" H 1800 7000 50  0001 C CNN "Source"
-F 5 "eeprom-so8w-W25Q" H -6100 -950 50  0001 C CNN "Key"
-	1    1800 7000
-	-1   0    0    -1
-$EndComp
 Wire Wire Line
 	3000 5300 3000 5500
@@
 L pkl_device:pkl_R4_Small R9
 U 2 1 5AB5B376
-P 10900 4500
-F 0 "R9" V 10850 4250 50  0000 L CNN
-F 1 "10k" V 10950 4250 50  0000 L CNN
-F 2 "pkl_dipol:R_Array_Convex_4x0402" H 10900 4500 60  0001 C CNN
-F 3 "" H 10900 4500 60  0000 C CNN
-F 4 "ANY" H 10900 4500 50  0001 C CNN "Source"
-F 5 "res-0402cv-array-4-10k" H 2200 -2900 50  0001 C CNN "Key"
-	2    10900 4500
+P 3000 5600
+F 0 "R9" V 2950 5350 50  0000 L CNN
+F 1 "10k" V 2950 5700 50  0000 L CNN
+F 2 "pkl_dipol:R_Array_Convex_4x0402" H 3000 5600 60  0001 C CNN
+F 3 "" H 3000 5600 60  0000 C CNN
+F 4 "ANY" H 3000 5600 50  0001 C CNN "Source"
+F 5 "res-0402cv-array-4-10k" H -5700 -1800 50  0001 C CNN "Key"
+	2    3000 5600
 	1    0    0    -1
 $EndComp
@@
 	2400 6400 2500 6400
 Text Notes 1900 5000 0    50   ~ 0
-JP3: Remove jumper when only programming iCE\nReplace jumper for programming Flash and for normal operation
+JP3: Cut jumper when only programming iCE\nConnect jumper for programming Flash and for normal operation
 $Comp
 L pkl_memory:VTI7064 U4
@@
 U 4 1 5ABF66A6
 P 2800 5600
-F 0 "R9" V 2750 5350 50  0000 L CNN
-F 1 "10k" V 2750 5700 50  0000 L CNN
+F 0 "R9" V 2850 5850 50  0000 R CNN
+F 1 "10k" V 2850 5500 50  0000 R CNN
 F 2 "pkl_dipol:R_Array_Convex_4x0402" H 2800 5600 60  0001 C CNN
 F 3 "" H 2800 5600 60  0000 C CNN
@@
 F 5 "res-0402cv-array-4-10k" H -6100 -1800 50  0001 C CNN "Key"
 	4    2800 5600
-	1    0    0    -1
+	-1   0    0    1
 $EndComp
 $Comp
 L pkl_device:pkl_R4_Small R9
 U 3 1 5ABF6624
-P 3000 5600
-F 0 "R9" V 2950 5350 50  0000 L CNN
-F 1 "10k" V 2950 5700 50  0000 L CNN
-F 2 "pkl_dipol:R_Array_Convex_4x0402" H 3000 5600 60  0001 C CNN
-F 3 "" H 3000 5600 60  0000 C CNN
-F 4 "ANY" H 3000 5600 50  0001 C CNN "Source"
-F 5 "res-0402cv-array-4-10k" H -5600 -1800 50  0001 C CNN "Key"
-	3    3000 5600
-	1    0    0    -1
+P 10900 4500
+F 0 "R9" V 10950 4750 50  0000 R CNN
+F 1 "10k" V 10850 4750 50  0000 R CNN
+F 2 "pkl_dipol:R_Array_Convex_4x0402" H 10900 4500 60  0001 C CNN
+F 3 "" H 10900 4500 60  0000 C CNN
+F 4 "ANY" H 10900 4500 50  0001 C CNN "Source"
+F 5 "res-0402cv-array-4-10k" H 2300 -2900 50  0001 C CNN "Key"
+	3    10900 4500
+	-1   0    0    1
 $EndComp
 Wire Wire Line
@@
 	10200 4600 10300 4600
 $Comp
+L pkl_memory:W25Q U5
+U 1 1 5A9D24AF
+P 1800 7000
+F 0 "U5" H 1800 7400 50  0000 C CNN
+F 1 "W25Q128JVxxM" H 1800 7300 50  0000 C CNN
+F 2 "Package_SON:WSON-8-1EP_6x5mm_P1.27mm_EP3.4x4.3mm" H 1800 7000 50  0001 C CNN
+F 3 "" H 1800 7000 50  0001 C CNN
+F 4 "ANY" H 1800 7000 50  0001 C CNN "Source"
+F 5 "eeprom-so8w-W25Q" H -6100 -950 50  0001 C CNN "Key"
+	1    1800 7000
+	-1   0    0    -1
+$EndComp
+Text Notes 5900 7200 0    50   ~ 0
+Main In Secondary Out
+Text Notes 5900 7300 0    50   ~ 0
+Main Out Secondary In
+Text Notes 5900 7100 0    50   ~ 0
+Serial Clock
+Wire Wire Line
+	5300 7500 5200 7500
+Text Label 5300 7500 0    50   ~ 0
+SPI_~WP~-IO2
+$Comp
+L Connector_Generic:Conn_01x01 P40
+U 1 1 5F31CDE3
+P 5000 7400
+F 0 "P40" H 5080 7396 50  0000 L CNN
+F 1 "IO3" H 5080 7351 50  0001 L CNN
+F 2 "pkl_pads:PAD_SMD_R_1x1" H 5000 7400 50  0001 C CNN
+F 3 "~" H 5000 7400 50  0001 C CNN
+	1    5000 7400
+	-1   0    0    -1
+$EndComp
+$Comp
+L Connector_Generic:Conn_01x01 P39
+U 1 1 5F31B48D
+P 5000 7300
+F 0 "P39" H 5080 7296 50  0000 L CNN
+F 1 "MOSI" H 5080 7251 50  0001 L CNN
+F 2 "pkl_pin_headers:Pin_Header_Straight_Round_1x01" H 5000 7300 50  0001 C CNN
+F 3 "~" H 5000 7300 50  0001 C CNN
+	1    5000 7300
+	-1   0    0    -1
+$EndComp
+$Comp
+L Connector_Generic:Conn_01x01 P38
+U 1 1 5F31B224
+P 5000 7200
+F 0 "P38" H 5080 7196 50  0000 L CNN
+F 1 "MISO" H 5080 7151 50  0001 L CNN
+F 2 "pkl_pin_headers:Pin_Header_Straight_Round_1x01" H 5000 7200 50  0001 C CNN
+F 3 "~" H 5000 7200 50  0001 C CNN
+	1    5000 7200
+	-1   0    0    -1
+$EndComp
+$Comp
+L Connector_Generic:Conn_01x01 P37
+U 1 1 5F31B068
+P 5000 7100
+F 0 "P37" H 5080 7096 50  0000 L CNN
+F 1 "SCK" H 5080 7051 50  0001 L CNN
+F 2 "pkl_pin_headers:Pin_Header_Straight_Round_1x01" H 5000 7100 50  0001 C CNN
+F 3 "~" H 5000 7100 50  0001 C CNN
+	1    5000 7100
+	-1   0    0    -1
+$EndComp
+$Comp
+L Connector_Generic:Conn_01x01 P36
+U 1 1 5F31319B
+P 5000 7000
+F 0 "P36" H 5080 6996 50  0000 L CNN
+F 1 "CS" H 5080 6951 50  0001 L CNN
+F 2 "pkl_pin_headers:Pin_Header_Straight_Round_1x01" H 5000 7000 50  0001 C CNN
+F 3 "~" H 5000 7000 50  0001 C CNN
+	1    5000 7000
+	-1   0    0    -1
+$EndComp
+Wire Wire Line
+	5300 7300 5200 7300
+Wire Wire Line
+	5300 7200 5200 7200
+Wire Wire Line
+	5200 7400 5300 7400
+Wire Wire Line
+	5200 7100 5300 7100
+Wire Wire Line
+	5200 7000 5300 7000
+Text Label 5300 7400 0    50   ~ 0
+SPI_~HLD~-IO3
+Text Label 5300 7300 0    50   ~ 0
+SPI_MOSI-IO0
+Text Label 5300 7200 0    50   ~ 0
+SPI_MISO-IO1
+Text Label 5300 7100 0    50   ~ 0
+SPI_SCK
+Text Label 5300 7000 0    50   ~ 0
+SPI_~CS
+$Comp
 L Connector_Generic:Conn_01x01 P41
 U 1 1 5F35ED22
-P 5500 7500
-F 0 "P41" H 5580 7496 50  0000 L CNN
-F 1 "IO2" H 5580 7451 50  0001 L CNN
-F 2 "pkl_pads:PAD_SMD_R_1x1" H 5500 7500 50  0001 C CNN
-F 3 "~" H 5500 7500 50  0001 C CNN
-	1    5500 7500
+P 5000 7500
+F 0 "P41" H 5080 7496 50  0000 L CNN
+F 1 "IO2" H 5080 7451 50  0001 L CNN
+F 2 "pkl_pads:PAD_SMD_R_1x1" H 5000 7500 50  0001 C CNN
+F 3 "~" H 5000 7500 50  0001 C CNN
+	1    5000 7500
 	-1   0    0    -1
 $EndComp
-Text Label 5800 7000 0    50   ~ 0
-SPI_~CS
-Text Label 5800 7100 0    50   ~ 0
-SPI_SCK
-Text Label 5800 7200 0    50   ~ 0
-SPI_MISO-IO1
-Text Label 5800 7300 0    50   ~ 0
-SPI_MOSI-IO0
-Text Label 5800 7400 0    50   ~ 0
-SPI_~HLD~-IO3
-Wire Wire Line
-	5700 7000 5800 7000
-Wire Wire Line
-	5700 7100 5800 7100
-Wire Wire Line
-	5700 7400 5800 7400
-Wire Wire Line
-	5800 7200 5700 7200
-Wire Wire Line
-	5800 7300 5700 7300
-$Comp
-L Connector_Generic:Conn_01x01 P36
-U 1 1 5F31319B
-P 5500 7000
-F 0 "P36" H 5580 6996 50  0000 L CNN
-F 1 "CS" H 5580 6951 50  0001 L CNN
-F 2 "pkl_pin_headers:Pin_Header_Straight_Round_1x01" H 5500 7000 50  0001 C CNN
-F 3 "~" H 5500 7000 50  0001 C CNN
-	1    5500 7000
-	-1   0    0    -1
-$EndComp
-$Comp
-L Connector_Generic:Conn_01x01 P37
-U 1 1 5F31B068
-P 5500 7100
-F 0 "P37" H 5580 7096 50  0000 L CNN
-F 1 "SCK" H 5580 7051 50  0001 L CNN
-F 2 "pkl_pin_headers:Pin_Header_Straight_Round_1x01" H 5500 7100 50  0001 C CNN
-F 3 "~" H 5500 7100 50  0001 C CNN
-	1    5500 7100
-	-1   0    0    -1
-$EndComp
-$Comp
-L Connector_Generic:Conn_01x01 P38
-U 1 1 5F31B224
-P 5500 7200
-F 0 "P38" H 5580 7196 50  0000 L CNN
-F 1 "MISO" H 5580 7151 50  0001 L CNN
-F 2 "pkl_pin_headers:Pin_Header_Straight_Round_1x01" H 5500 7200 50  0001 C CNN
-F 3 "~" H 5500 7200 50  0001 C CNN
-	1    5500 7200
-	-1   0    0    -1
-$EndComp
-$Comp
-L Connector_Generic:Conn_01x01 P39
-U 1 1 5F31B48D
-P 5500 7300
-F 0 "P39" H 5580 7296 50  0000 L CNN
-F 1 "MOSI" H 5580 7251 50  0001 L CNN
-F 2 "pkl_pin_headers:Pin_Header_Straight_Round_1x01" H 5500 7300 50  0001 C CNN
-F 3 "~" H 5500 7300 50  0001 C CNN
-	1    5500 7300
-	-1   0    0    -1
-$EndComp
-$Comp
-L Connector_Generic:Conn_01x01 P40
-U 1 1 5F31CDE3
-P 5500 7400
-F 0 "P40" H 5580 7396 50  0000 L CNN
-F 1 "IO3" H 5580 7351 50  0001 L CNN
-F 2 "pkl_pads:PAD_SMD_R_1x1" H 5500 7400 50  0001 C CNN
-F 3 "~" H 5500 7400 50  0001 C CNN
-	1    5500 7400
-	-1   0    0    -1
-$EndComp
-Text Label 5800 7500 0    50   ~ 0
-SPI_~WP~-IO2
-Wire Wire Line
-	5800 7500 5700 7500
-Text Notes 6300 3150 0    50   ~ 0
-SPI Terminology:\nMOSI - Main Out Secondary In\nMISO - Main In Secondary Out\nSCK  - Serial Clock\nCS   - Chip Select
+Text Notes 5900 7000 0    50   ~ 0
+Chip Select
+Text Notes 5900 7400 0    50   ~ 0
+Hold
+Text Notes 5900 7500 0    50   ~ 0
+Write Protect
 $EndSCHEMATC
