File: hardware/bitsy-v1.1a/icebreaker-bitsy.sch (KiCad schematic (older format))
At the start: 95 parts, among them J1 USB_C, P0 0, P1 1, P10 10, P11 11, P12 12, P13 13, P14 14, P15 15, P16 16, P17 17, P18 18, P19 19, P2 2, P20 20, P21 21, P22 22, P23 23, P24 GND, P25 GND, P26 GND, P27 3V3, P28 3V3, P29 VIN, P3 3, P30 CDONE, P31 CRESET, P32 UP, P33 UP, P34 UP, P35 UP, P36 CS, P37 SCK, P38 MISO, P39 MOSI, P4 4, P40 IO3, P41 IO2, P5 5, P6 6, P7 7, P8 8, P9 9, SW1 TACT, U1 USBLC6-2, U2 TLV75533PDRV, U3 TLV75512PDRV, U4 LY68L6400, U5 W25Q128JVxxM, U6 ICE40UP5K-SG48, X1 12MHz

Commit message: Finish up some more TODOs
- change LED resistor values
- update interactive BOM
- update PDFs
- clean up PCB planes & comments
Other:
- moved on the sheet: P27, P28, P29
Changed lines of the file:
@@
 encoding utf-8
 Sheet 1 1
-Title "iCEBreaker-bitsy"
-Date "2020-08-04"
+Title "iCEBreaker Bitsy"
+Date "2020-08-05"
 Rev "v1.1a"
 Comp "1BitSquared"
@@
 $EndComp
 $Comp
-L power:+3V3 #PWR0128
-U 1 1 5F6139CB
-P 7500 5800
-F 0 "#PWR0128" H 7500 5650 50  0001 C CNN
-F 1 "+3V3" H 7500 5950 50  0000 C CNN
-F 2 "" H 7500 5800 50  0001 C CNN
-F 3 "" H 7500 5800 50  0001 C CNN
-	1    7500 5800
-	1    0    0    -1
-$EndComp
-$Comp
 L Connector_Generic:Conn_01x01 P26
 U 1 1 5B1A640B
@@
 	0    -1   -1   0
 $EndComp
-$Comp
-L Connector_Generic:Conn_01x01 P27
-U 1 1 5B1151BE
-P 7200 6000
-F 0 "P27" V 7300 6000 50  0000 C CNN
-F 1 "3V3" H 7280 5949 50  0001 L CNN
-F 2 "pkl_pin_headers:Pin_Header_Straight_Round_1x01_Castellated" H 7200 6000 50  0001 C CNN
-F 3 "~" H 7200 6000 50  0001 C CNN
-F 4 "ANY" H 7200 6000 50  0001 C CNN "Source"
-	1    7200 6000
-	0    1    1    0
-$EndComp
-$Comp
-L Connector_Generic:Conn_01x01 P28
-U 1 1 5B14536A
-P 7500 6000
-F 0 "P28" V 7600 6000 50  0000 C CNN
-F 1 "3V3" H 7580 5949 50  0001 L CNN
-F 2 "pkl_pin_headers:Pin_Header_Straight_Round_1x01_Castellated" H 7500 6000 50  0001 C CNN
-F 3 "~" H 7500 6000 50  0001 C CNN
-F 4 "ANY" H 7500 6000 50  0001 C CNN "Source"
-	1    7500 6000
-	0    1    1    0
-$EndComp
-$Comp
-L Connector_Generic:Conn_01x01 P29
-U 1 1 5B1A6195
-P 7800 6000
-F 0 "P29" V 7900 6000 50  0000 C CNN
-F 1 "VIN" H 7880 5949 50  0001 L CNN
-F 2 "pkl_pin_headers:Pin_Header_Straight_Round_1x01_Castellated" H 7800 6000 50  0001 C CNN
-F 3 "~" H 7800 6000 50  0001 C CNN
-F 4 "ANY" H 7800 6000 50  0001 C CNN "Source"
-	1    7800 6000
-	0    1    1    0
-$EndComp
-$Comp
-L power:+3V3 #PWR04
-U 1 1 5B1A5E3B
-P 7200 5800
-F 0 "#PWR04" H 7200 5650 50  0001 C CNN
-F 1 "+3V3" H 7200 5950 50  0000 C CNN
-F 2 "" H 7200 5800 50  0001 C CNN
-F 3 "" H 7200 5800 50  0001 C CNN
-	1    7200 5800
-	1    0    0    -1
-$EndComp
 Wire Notes Line
 	8000 6400 6100 6400
 Wire Notes Line
 	6100 6400 6100 5500
-$Comp
-L pkl_power:VIN #PWR0109
-U 1 1 5F45B3FF
-P 7800 5800
-F 0 "#PWR0109" H 7800 5650 50  0001 C CNN
-F 1 "VIN" H 7800 5950 50  0000 C CNN
-F 2 "" H 7800 5800 50  0001 C CNN
-F 3 "" H 7800 5800 50  0001 C CNN
-	1    7800 5800
-	1    0    0    -1
-$EndComp
 Wire Notes Line
 	8000 5500 8000 6400
@@
 Text Notes 5900 7500 0    50   ~ 0
 Write Protect
+$Comp
+L pkl_power:VIN #PWR0109
+U 1 1 5F45B3FF
+P 7800 5900
+F 0 "#PWR0109" H 7800 5750 50  0001 C CNN
+F 1 "VIN" H 7800 6050 50  0000 C CNN
+F 2 "" H 7800 5900 50  0001 C CNN
+F 3 "" H 7800 5900 50  0001 C CNN
+	1    7800 5900
+	1    0    0    -1
+$EndComp
+$Comp
+L power:+3V3 #PWR04
+U 1 1 5B1A5E3B
+P 7200 5900
+F 0 "#PWR04" H 7200 5750 50  0001 C CNN
+F 1 "+3V3" H 7200 6050 50  0000 C CNN
+F 2 "" H 7200 5900 50  0001 C CNN
+F 3 "" H 7200 5900 50  0001 C CNN
+	1    7200 5900
+	1    0    0    -1
+$EndComp
+$Comp
+L Connector_Generic:Conn_01x01 P29
+U 1 1 5B1A6195
+P 7800 6100
+F 0 "P29" V 7900 6100 50  0000 C CNN
+F 1 "VIN" H 7880 6049 50  0001 L CNN
+F 2 "pkl_pin_headers:Pin_Header_Straight_Round_1x01_Castellated" H 7800 6100 50  0001 C CNN
+F 3 "~" H 7800 6100 50  0001 C CNN
+F 4 "ANY" H 7800 6100 50  0001 C CNN "Source"
+	1    7800 6100
+	0    1    1    0
+$EndComp
+$Comp
+L Connector_Generic:Conn_01x01 P28
+U 1 1 5B14536A
+P 7500 6100
+F 0 "P28" V 7600 6100 50  0000 C CNN
+F 1 "3V3" H 7580 6049 50  0001 L CNN
+F 2 "pkl_pin_headers:Pin_Header_Straight_Round_1x01_Castellated" H 7500 6100 50  0001 C CNN
+F 3 "~" H 7500 6100 50  0001 C CNN
+F 4 "ANY" H 7500 6100 50  0001 C CNN "Source"
+	1    7500 6100
+	0    1    1    0
+$EndComp
+$Comp
+L Connector_Generic:Conn_01x01 P27
+U 1 1 5B1151BE
+P 7200 6100
+F 0 "P27" V 7300 6100 50  0000 C CNN
+F 1 "3V3" H 7280 6049 50  0001 L CNN
+F 2 "pkl_pin_headers:Pin_Header_Straight_Round_1x01_Castellated" H 7200 6100 50  0001 C CNN
+F 3 "~" H 7200 6100 50  0001 C CNN
+F 4 "ANY" H 7200 6100 50  0001 C CNN "Source"
+	1    7200 6100
+	0    1    1    0
+$EndComp
+$Comp
+L power:+3V3 #PWR0128
+U 1 1 5F6139CB
+P 7500 5900
+F 0 "#PWR0128" H 7500 5750 50  0001 C CNN
+F 1 "+3V3" H 7500 6050 50  0000 C CNN
+F 2 "" H 7500 5900 50  0001 C CNN
+F 3 "" H 7500 5900 50  0001 C CNN
+	1    7500 5900
+	1    0    0    -1
+$EndComp
 $EndSCHEMATC

Commit message: icebitsy v1.1a: Updated bom keys.
Parts:
- C8: Key cap-cer-0402-10n -> cap-cer-0402-100n
- J1: Key (none) -> conn-smd-usb-c-2
- R11, R12: Key res-0402-330 -> res-0402-2k2
- R2, R3: Key res-0402-1m -> res-0402-5k1
- U2: Key (none) -> vreg-dfn6-1v2-tlv75533
- U3: value TLV75512PDRV -> TLV73312PDRV; Key (none) -> vreg-dfn6-1v2-tlv73312
- U5: Key eeprom-so8w-W25Q -> eeprom-wson8-w25q128
- X1: Key (none) -> osc-smd2520-12mhz
Changed lines of the file:
@@
 F 3 "" H 5600 2700 60  0000 C CNN
 F 4 "ANY" H 5600 2700 50  0001 C CNN "Source"
-F 5 "res-0402-330" H -7300 -6200 50  0001 C CNN "Key"
+F 5 "res-0402-2k2" H -7300 -6200 50  0001 C CNN "Key"
 	1    5600 2700
 	0    -1   -1   0
@@
 F 3 "" H 5600 3100 60  0000 C CNN
 F 4 "ANY" H 5600 3100 50  0001 C CNN "Source"
-F 5 "res-0402-330" H -7300 -5500 50  0001 C CNN "Key"
+F 5 "res-0402-2k2" H -7300 -5500 50  0001 C CNN "Key"
 	1    5600 3100
 	0    -1   -1   0
@@
 F 3 "" H 2200 1400 60  0000 C CNN
 F 4 "ANY" H 2200 1400 50  0001 C CNN "Source"
-F 5 "res-0402-1m" H 400 -3450 50  0001 C CNN "Key"
+F 5 "res-0402-5k1" H 400 -3450 50  0001 C CNN "Key"
 	1    2200 1400
 	0    1    1    0
@@
 F 3 "" H 2200 1500 60  0000 C CNN
 F 4 "ANY" H 2200 1500 50  0001 C CNN "Source"
-F 5 "res-0402-1m" H 400 -3350 50  0001 C CNN "Key"
+F 5 "res-0402-5k1" H 400 -3350 50  0001 C CNN "Key"
 	1    2200 1500
 	0    1    1    0
@@
 F 2 "pkl_connectors:USB_C_Receptacle_HRO_TYPE-C-31-M-12" H 1350 1800 50  0001 C CNN
 F 3 "https://www.usb.org/sites/default/files/documents/usb_type-c.zip" H 1350 1800 50  0001 C CNN
+F 4 "conn-smd-usb-c-2" H 1200 1800 50  0001 C CNN "Key"
 	1    1200 1800
 	1    0    0    -1
@@
 P 3800 4000
 F 0 "U3" H 3800 4342 50  0000 C CNN
-F 1 "TLV75512PDRV" H 3800 4251 50  0000 C CNN
+F 1 "TLV73312PDRV" H 3800 4251 50  0000 C CNN
 F 2 "Package_SON:WSON-6-1EP_2x2mm_P0.65mm_EP1x1.6mm" H 3800 4325 50  0001 C CIN
 F 3 "http://www.ti.com/lit/ds/symlink/tlv755p.pdf" H 3800 4050 50  0001 C CNN
+F 4 "vreg-dfn6-1v2-tlv73312" H 3800 4000 50  0001 C CNN "Key"
 	1    3800 4000
 	1    0    0    -1
@@
 F 2 "pkl_dipol:C_0402" H 7392 4907 60  0001 L CNN
 F 3 "" H 7300 5000 60  0000 C CNN
-F 4 "cap-cer-0402-10n" H 7300 5000 50  0001 C CNN "Key"
+F 4 "cap-cer-0402-100n" H 7300 5000 50  0001 C CNN "Key"
 F 5 "ANY" H 7300 5000 50  0001 C CNN "Source"
 	1    7300 5000
@@
 F 2 "Package_SON:WSON-6-1EP_2x2mm_P0.65mm_EP1x1.6mm" H 2300 4325 50  0001 C CIN
 F 3 "http://www.ti.com/lit/ds/symlink/tlv755p.pdf" H 2300 4050 50  0001 C CNN
+F 4 "vreg-dfn6-1v2-tlv75533" H 2300 4000 50  0001 C CNN "Key"
 	1    2300 4000
 	1    0    0    -1
@@
 F 2 "pkl_misc:Oscillator_SMD_SCTF_S2DXX-4Pin_2.5x2.0mm" H 6100 5250 50  0001 C CNN
 F 3 "" H 5300 5600 50  0001 C CNN
+F 4 "osc-smd2520-12mhz" H 5400 5600 50  0001 C CNN "Key"
 	1    5400 5600
 	1    0    0    -1
@@
 F 3 "" H 1800 7000 50  0001 C CNN
 F 4 "ANY" H 1800 7000 50  0001 C CNN "Source"
-F 5 "eeprom-so8w-W25Q" H -6100 -950 50  0001 C CNN "Key"
+F 5 "eeprom-wson8-w25q128" H -6100 -950 50  0001 C CNN "Key"
 	1    1800 7000
 	-1   0    0    -1

Commit message: icebitsy v1.1a: Corrected oscillator bom key.
Parts:
- X1: Key osc-smd2520-12mhz -> xtal-smd2520-12mhz-osc
Changed lines of the file:
@@
 F 2 "pkl_misc:Oscillator_SMD_SCTF_S2DXX-4Pin_2.5x2.0mm" H 6100 5250 50  0001 C CNN
 F 3 "" H 5300 5600 50  0001 C CNN
-F 4 "osc-smd2520-12mhz" H 5400 5600 50  0001 C CNN "Key"
+F 4 "xtal-smd2520-12mhz-osc" H 5400 5600 50  0001 C CNN "Key"
 	1    5400 5600
 	1    0    0    -1

Commit message: icebitsy v1.1a: Corrected the ice40up5k bom key.
Parts:
- U6: Key ic-ice5lp4k-sg48 -> ic-ice40up5k-sg48
Changed lines of the file:
@@
 F 3 "" H 10900 3300 50  0001 C CNN
 F 4 "ANY" H 8600 3100 50  0001 C CNN "Source"
-F 5 "ic-ice5lp4k-sg48" H -1000 -1100 50  0001 C CNN "Key"
+F 5 "ic-ice40up5k-sg48" H -1000 -1100 50  0001 C CNN "Key"
 	1    8600 3100
 	1    0    0    -1
