File: hardware/bitsy-v1.1a/icebreaker-bitsy.sch (KiCad schematic (older format))
At the start: 95 parts, among them J1 USB_C, P0 0, P1 1, P10 10, P11 11, P12 12, P13 13, P14 14, P15 15, P16 16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

Commit message: icebitsy v1.1a: Corrected RGB LED bom ID.
Parts:
- D4: Key led-1010-rgb -> led-2020-rgb
Changed lines of the file:
@@
 F 2 "pkl_led:LED_TRI_2020" H 5500 4150 50  0001 C CNN
 F 3 "~" H 5500 4150 50  0001 C CNN
-F 4 "led-1010-rgb" H 5500 4200 50  0001 C CNN "Key"
+F 4 "led-2020-rgb" H 5500 4200 50  0001 C CNN "Key"
 	1    5500 4200
 	1    0    0    -1
