File: hardware/bitsy-v1.1b/icebreaker-bitsy.kicad_pcb (KiCad board)
At the start: 4 copper layers, 35.6 x 18 mm, 99 parts, among them J1 USB_C, P0 0, P1 1, P10 10, P11 11, P12 12, P13 13, P14 14, P15 15, P16 16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

Commit message: icebitsy V1.1b: Removed solder stop expansion setting.
Other:
- rule pad_to_mask_clearance: 0.05 -> 0
